Commit message: Adding more comments to the robot description of Oberon and changing some joint dynamics configurations.
Signed-off-by: Musa Morena Marcusso Manhães <Musa.Marcusso@de.bosch.com>

File: uuv_manipulators/oberon/oberon_description/urdf/dummy_gripper.xacro (robot description, xacro)
@@ -1,4 +1,4 @@
 <?xml version="1.0"?>
-<!-- Oberon-7P Schilling Robotics Manipulator Dummy Gripper
+<!-- Oberon-7P Dummy Gripper (inspired on the Orion 7P Schilling Robotics Manipulator)
     Meshes and parameters a courtesy of Deutsche Forschungszentrum für
     Künstliche Intelligenz GmbH (DFKI)

File: uuv_manipulators/oberon/oberon_description/urdf/parallel_gripper.xacro (robot description, xacro)
@@ -12,5 +12,5 @@
      limitations under the License.
 -->
-<!-- Oberon-7P Schilling Robotics Manipulator Parallel Gripper -->
+<!-- Oberon-7P Parallel Gripper (inspired on the Orion 7P Schilling Robotics Manipulator) -->
 <robot xmlns:xacro="http://www.ros.org/wiki/xacro">
     <xacro:property name="mass_gripper" value="3.96" /> <!-- mass of Gripper (kg) - 54kg*0,001422/0,019395 = 3,96 kg -->
@@ -107,5 +107,5 @@
             <origin xyz="0.0 -0.028 0.05" rpy="0 ${-pi*0.5} 0"/>
             <axis xyz="0 0 1"/>
-            <limit effort="${gripper_effort}" lower="${-pi*0.25}" upper="0" velocity="${gripper_velocity}"/>
+            <limit effort="${gripper_effort}" lower="${-pi*0.3333}" upper="0" velocity="${gripper_velocity}"/>
             <dynamics damping="5" friction="10"/>
         </joint>
@@ -169,5 +169,5 @@
             <origin xyz="0.0 0.028 0.05" rpy="0 ${-pi*0.5} ${pi}"/>
             <axis xyz="0 0 1"/>
-            <limit effort="${gripper_effort}" lower="${-pi*0.25}" upper="0" velocity="${gripper_velocity}"/>
+            <limit effort="${gripper_effort}" lower="${-pi*0.3333}" upper="0" velocity="${gripper_velocity}"/>
             <dynamics damping="5" friction="10"/>
         </joint>
@@ -215,15 +215,4 @@
             <!-- <maxContacts>5</maxContacts> -->
         </gazebo>
-        <!-- Setting up mimic joints -->
-        <gazebo>
-          <plugin name="mimic_finger" filename="libgazebo_ros_mimic_joints.so">
-            <robotNamespace>${namespace}</robotNamespace>
-            <joint>${namespace}/finger_left_joint</joint>
-            <mimicJoint>${namespace}/finger_right_joint</mimicJoint>
-            <kp>60</kp>
-            <kd>5</kd>
-            <ki>1</ki>
-          </plugin>
-        </gazebo>
     </xacro:macro>
 </robot>

File: uuv_manipulators/oberon/oberon_description/urdf/serial_arm.xacro (robot description, xacro)
@@ -1,4 +1,4 @@
 <?xml version="1.0"?>
-<!-- Oberon-7P Schilling Robotics Manipulator
+<!-- Oberon-7P Manipulator (inspired on the Orion 7P Schilling Robotics Manipulator)
      Meshes and parameters a courtesy of Deutsche Forschungszentrum für
      Künstliche Intelligenz GmbH (DFKI)
@@ -290,11 +290,10 @@
       <limit lower="-1.6406094968746698" upper="0.4537856055185257" velocity=".26" effort="10000"/>
     </joint>
-    <joint name="${namespace}/wrist" type="revolute">
+    <joint name="${namespace}/wrist" type="continuous">
       <parent link="${namespace}/wrist_2"/>
       <child link="${namespace}/end_effector"/>
       <origin xyz="0.232 0 0" rpy="0 0 0"/>
       <axis xyz="1 0 0"/>
-      <dynamics damping="15" friction="40"/>
-      <limit lower="-0.38397243543875248" upper="5.8817595792208905" velocity=".26" effort="5"/>
+      <dynamics damping="10" friction="60"/>
     </joint>
     <!-- Transmissions -->
