Commit message: replace collision meshes with primitives
modify joint parameters as suggested here:
http://answers.gazebosim.org/question/13700/object-slips-out-of-the-gripper-after-jitters/

Signed-off-by: Sebastian Scherer <Sebastian.Scherer2@de.bosch.com>

File: uuv_manipulators/oberon/oberon_description/urdf/parallel_gripper.xacro (robot description, xacro)
@@ -14,4 +14,5 @@
 <!-- Oberon-7P Parallel Gripper (inspired on the Orion 7P Schilling Robotics Manipulator) -->
 <robot xmlns:xacro="http://www.ros.org/wiki/xacro">
+    <xacro:property name="use_mesh_file" value="false" />
     <xacro:property name="mass_gripper" value="3.96" /> <!-- mass of Gripper (kg) - 54kg*0,001422/0,019395 = 3,96 kg -->
     <xacro:property name="gripper_effort" value="200" />
@@ -25,12 +26,12 @@
     <!-- Properties for the finger -->
     <xacro:property name="gripper_finger_mesh" value="file://$(find oberon_description)/meshes/grippers/parallel/oberon_finger"/>
-    <xacro:property name="gripper_finger_x" value="0.15"/>
-    <xacro:property name="gripper_finger_y" value="0.056"/>
-    <xacro:property name="gripper_finger_z" value="0.03"/>
+    <xacro:property name="gripper_finger_x" value="0.10"/>
+    <xacro:property name="gripper_finger_y" value="0.02"/>
+    <xacro:property name="gripper_finger_z" value="0.05"/>
     <xacro:property name="gripper_finger_volume" value="${gripper_finger_x*gripper_finger_y*gripper_finger_z}"/>
     <!-- Properties of the tip -->
     <xacro:property name="gripper_tip_mesh" value="file://$(find oberon_description)/meshes/grippers/parallel/oberon_tip"/>
-    <xacro:property name="gripper_tip_x" value="0.1"/>
-    <xacro:property name="gripper_tip_y" value="0.05"/>
+    <xacro:property name="gripper_tip_x" value="0.04"/>
+    <xacro:property name="gripper_tip_y" value="0.1"/>
     <xacro:property name="gripper_tip_z" value="0.079999"/>
     <xacro:property name="gripper_tip_volume" value="${gripper_tip_x*gripper_tip_y*gripper_tip_z}"/>
@@ -65,8 +66,16 @@
         </visual>
         <collision>
+          <xacro:if value="${use_mesh_file}">
             <origin xyz="0 0 0" rpy="0 0 0"/>
             <geometry>
                 <mesh filename="${mesh}.stl" scale="1 1 1"/>
             </geometry>
+          </xacro:if>
+          <xacro:unless value="${use_mesh_file}">
+            <xacro:insert_block name="origin" />
+            <geometry>
+                <box size="${x} ${y} ${z}" />
+            </geometry>
+          </xacro:unless>
         </collision>
     </xacro:macro>
@@ -99,5 +108,5 @@
                                 z="${gripper_finger_z}"
                                 mesh="${gripper_finger_mesh}">
-                <origin xyz="0.054821 -0.00812 0.0" rpy="0 0 0"/>
+                <origin xyz="0.05 -0.01 0.0" rpy="0 0 0"/>
             </xacro:gripper_link>
         </link>
@@ -112,14 +121,13 @@
         <xacro:simple_transmission joint="${namespace}/finger_left_joint"/>
         <gazebo reference="${namespace}/finger_left">
-            <selfCollide>true</selfCollide>
-            <mu1>1000</mu1>
-            <mu2>1000</mu2>
-            <fdir1>0 0 1</fdir1>
-            <kp>1000000.0</kp>
-            <kd>10000.0</kd>
-            <!-- <maxVel>0.1</maxVel> -->
-            <!-- <minDepth>0.001</minDepth> -->
-            <!-- <maxContacts>5</maxContacts> -->
-        </gazebo>
+          <selfCollide>true</selfCollide>
+          <kp>1000000.0</kp>
+          <kd>1.0</kd>
+          <mu1>1.0</mu1>
+          <mu2>1.0</mu2>
+          <minDepth>0.001</minDepth>
+          <maxContacts>3</maxContacts>
+          <implicitSpringDamper>1</implicitSpringDamper>
+      </gazebo>
         <!-- ****************************************************************************************************** -->
         <!-- Left finger tip -->
@@ -130,5 +138,5 @@
                                 z="${gripper_tip_z}"
                                 mesh="${gripper_tip_mesh}">
-                <origin xyz="-0.035 0.015 0.0" rpy="0 0 0"/>
+                <origin xyz="0.015 -0.035 0.0" rpy="0 0 0"/>
             </xacro:gripper_link>
         </link>
@@ -144,12 +152,11 @@
         <gazebo reference="${namespace}/finger_tip_left">
             <selfCollide>true</selfCollide>
-            <mu1>1000</mu1>
-            <mu2>1000</mu2>
-            <fdir1>0 0 1</fdir1>
             <kp>1000000.0</kp>
-            <kd>10000.0</kd>
-            <!-- <maxVel>0.1</maxVel> -->
-            <!-- <minDepth>0.001</minDepth> -->
-            <!-- <maxContacts>5</maxContacts> -->
+            <kd>1.0</kd>
+            <mu1>1.0</mu1>
+            <mu2>1.0</mu2>
+            <minDepth>0.001</minDepth>
+            <maxContacts>3</maxContacts>
+            <implicitSpringDamper>1</implicitSpringDamper>
         </gazebo>
         <!-- ****************************************************************************************************** -->
@@ -161,5 +168,5 @@
                                 z="${gripper_finger_z}"
                                 mesh="${gripper_finger_mesh}">
-                <origin xyz="0.054821 -0.008120 0.0" rpy="0 0 0"/>
+                <origin xyz="0.05 -0.01 0.0" rpy="0 0 0"/>
             </xacro:gripper_link>
         </link>
@@ -175,12 +182,11 @@
         <gazebo reference="${namespace}/finger_right">
             <selfCollide>true</selfCollide>
-            <mu1>1000</mu1>
-            <mu2>1000</mu2>
-            <fdir1>0 0 1</fdir1>
             <kp>1000000.0</kp>
-            <kd>10000.0</kd>
-            <!-- <maxVel>0.1</maxVel> -->
-            <!-- <minDepth>0.001</minDepth> -->
-            <!-- <maxContacts>5</maxContacts> -->
+            <kd>1.0</kd>
+            <mu1>1.0</mu1>
+            <mu2>1.0</mu2>
+            <minDepth>0.001</minDepth>
+            <maxContacts>3</maxContacts>
+            <implicitSpringDamper>1</implicitSpringDamper>
         </gazebo>
         <!-- ****************************************************************************************************** -->
@@ -192,5 +198,5 @@
                                 z="${gripper_tip_z}"
                                 mesh="${gripper_tip_mesh}">
-                <origin xyz="-0.035 0.015 0.0" rpy="0 0 0"/>
+                <origin xyz="0.015 -0.035 0.0" rpy="0 0 0"/>
             </xacro:gripper_link>
         </link>
@@ -205,14 +211,13 @@
         <xacro:simple_transmission joint="${namespace}/finger_tip_right_joint"/>
         <gazebo reference="${namespace}/finger_tip_right">
-            <selfCollide>true</selfCollide>
-            <mu1>1000</mu1>
-            <mu2>1000</mu2>
-            <fdir1>0 0 1</fdir1>
-            <kp>1000000.0</kp>
-            <kd>10000.0</kd>
-            <!-- <maxVel>0.1</maxVel> -->
-            <!-- <minDepth>0.001</minDepth> -->
-            <!-- <maxContacts>5</maxContacts> -->
-        </gazebo>
+          <selfCollide>true</selfCollide>
+          <kp>1000000.0</kp>
+          <kd>1.0</kd>
+          <mu1>1.0</mu1>
+          <mu2>1.0</mu2>
+          <minDepth>0.001</minDepth>
+          <maxContacts>3</maxContacts>
+          <implicitSpringDamper>1</implicitSpringDamper>
+      </gazebo>
     </xacro:macro>
 </robot>

File: uuv_manipulators/oberon/oberon_description/urdf/serial_arm.gazebo.xacro (robot description, xacro)
@@ -25,4 +25,28 @@
   <gazebo reference="${namespace}/end_effector">
     <selfCollide>false</selfCollide>
+  </gazebo>
+  <gazebo reference="${namespace}/anchor">
+    <implicitSpringDamper>1</implicitSpringDamper>
+  </gazebo>
+  <gazebo reference="${namespace}/azimuth">
+    <implicitSpringDamper>1</implicitSpringDamper>
+  </gazebo>
+  <gazebo reference="${namespace}/shoulder">
+    <implicitSpringDamper>1</implicitSpringDamper>
+  </gazebo>
+  <gazebo reference="${namespace}/elbow">
+    <implicitSpringDamper>1</implicitSpringDamper>
+  </gazebo>
+  <gazebo reference="${namespace}/elbow_dummy">
+    <implicitSpringDamper>1</implicitSpringDamper>
+  </gazebo>
+  <gazebo reference="${namespace}/roll">
+    <implicitSpringDamper>1</implicitSpringDamper>
+  </gazebo>
+  <gazebo reference="${namespace}/pitch">
+    <implicitSpringDamper>1</implicitSpringDamper>
+  </gazebo>
+  <gazebo reference="${namespace}/wrist">
+    <implicitSpringDamper>1</implicitSpringDamper>
   </gazebo>
   <gazebo>

File: uuv_manipulators/oberon4/oberon4_description/urdf/serial_arm.gazebo.xacro (robot description, xacro)
@@ -34,4 +34,25 @@
   <gazebo reference="${namespace}/jaw_2">
     <selfCollide>false</selfCollide>
+  </gazebo>
+  <gazebo reference="${namespace}/anchor">
+    <implicitSpringDamper>1</implicitSpringDamper>
+  </gazebo>
+  <gazebo reference="${namespace}/azimuth">
+    <implicitSpringDamper>1</implicitSpringDamper>
+  </gazebo>
+  <gazebo reference="${namespace}/shoulder">
+    <implicitSpringDamper>1</implicitSpringDamper>
+  </gazebo>
+  <gazebo reference="${namespace}/wrist_joint">
+    <implicitSpringDamper>1</implicitSpringDamper>
+  </gazebo>
+  <gazebo reference="${namespace}/gripper_joint">
+    <implicitSpringDamper>1</implicitSpringDamper>
+  </gazebo>
+  <gazebo reference="${namespace}/jaw_2_joint">
+    <implicitSpringDamper>1</implicitSpringDamper>
+  </gazebo>
+  <gazebo reference="${namespace}/jaw_1_joint">
+    <implicitSpringDamper>1</implicitSpringDamper>
   </gazebo>
   <gazebo>

File: uuv_manipulators/oberon4/oberon4_description/urdf/serial_arm.xacro (robot description, xacro)
@@ -14,5 +14,5 @@
 <robot xmlns:xacro="http://www.ros.org/wiki/xacro">
   <!-- Constants for robot dimensions -->
-  <xacro:property name="use_mesh_file" value="true" />
+  <xacro:property name="use_mesh_file" value="false" />
   <xacro:property name="PI" value="3.1415926535897931"/>
   <xacro:property name="base_volume" value="0.002325" />
@@ -30,5 +30,5 @@
   <xacro:property name="arm_volume" value="0.001583" />
   <xacro:property name="arm_mass" value="5.193" />
-  <xacro:property name="arm_x" value="0.42303" />
+  <xacro:property name="arm_x" value="0.375" />
   <xacro:property name="arm_y" value="0.128467" />
   <xacro:property name="arm_z" value="0.166069" />
@@ -193,10 +193,38 @@
         </geometry>
       </visual>
-      <collision>
-        <origin xyz="0 0 0" rpy="0 0 0" />
+      <xacro:if value="${use_mesh_file}">
+      <collision>
+        <origin xyz="0 0 0" rpy="0 0 0"/>
         <geometry>
           <mesh filename="file://$(find oberon4_description)/meshes/Jaw.stl" scale="1 1 1" />
         </geometry>
       </collision>
+      </xacro:if>
+      <xacro:unless value="${use_mesh_file}">
+        <collision>
+          <origin xyz="0.08 0.035 -0.002" rpy="0 0 0" />
+          <geometry>
+            <box size="0.12 0.02 0.025"/>
+          </geometry>
+        </collision>
+        <collision>
+          <origin xyz="0.145 0.055 -0.002" rpy="0 0 0.7" />
+          <geometry>
+            <box size="0.07 0.015 0.025"/>
+          </geometry>
+        </collision>
+        <collision>
+          <origin xyz="0.08 0.035 -0.07" rpy="0 0 0" />
+          <geometry>
+            <box size="0.12 0.02 0.025"/>
+          </geometry>
+        </collision>
+        <collision>
+          <origin xyz="0.145 0.055 -0.07" rpy="0 0 0.7" />
+          <geometry>
+            <box size="0.07 0.015 0.025"/>
+          </geometry>
+        </collision>
+      </xacro:unless>
     </link>
     <!-- Jaw 2 link  -->
@@ -215,10 +243,38 @@
         </geometry>
       </visual>
-      <collision>
-        <origin xyz="0 0 0" rpy="0 0 0" />
+      <xacro:if value="${use_mesh_file}">
+      <collision>
+        <origin xyz="0 0 0" rpy="0 0 0"/>
         <geometry>
           <mesh filename="file://$(find oberon4_description)/meshes/Jaw.stl" scale="1 1 1" />
         </geometry>
       </collision>
+      </xacro:if>
+      <xacro:unless value="${use_mesh_file}">
+      <collision>
+        <origin xyz="0.08 0.035 -0.002" rpy="0 0 0" />
+        <geometry>
+          <box size="0.12 0.02 0.025"/>
+        </geometry>
+      </collision>
+      <collision>
+        <origin xyz="0.145 0.055 -0.002" rpy="0 0 0.7" />
+        <geometry>
+          <box size="0.07 0.015 0.025"/>
+        </geometry>
+      </collision>
+      <collision>
+        <origin xyz="0.08 0.035 -0.07" rpy="0 0 0" />
+        <geometry>
+          <box size="0.12 0.02 0.025"/>
+        </geometry>
+      </collision>
+      <collision>
+        <origin xyz="0.145 0.055 -0.07" rpy="0 0 0.7" />
+        <geometry>
+          <box size="0.07 0.015 0.025"/>
+        </geometry>
+      </collision>
+    </xacro:unless>
     </link>
     <!-- All the joints -->
