Commit message: Modifying launch files and adding new demos with a joystick mapping for the Logitech Extreme 3D Pro.
Signed-off-by: Musa Morena Marcusso Manhães <Musa.Marcusso@de.bosch.com>

File: uuv_manipulators/oberon/oberon_description/urdf/serial_arm.xacro (robot description, xacro)
@@ -249,5 +249,5 @@
       <child link="${namespace}/shoulder_link"/>
       <axis xyz="0 0 1"/>
-      <dynamics damping="15" friction="40"/>
+      <dynamics damping="20" friction="50"/>
       <limit lower="-1.0471975511965976" upper="1.0471975511965976" velocity="0.17" effort="10000"/>
     </joint>
@@ -257,5 +257,5 @@
         <origin xyz="0.07 0.0 0.028" rpy="0 0 0"/>
         <axis xyz="0 -1 0"/>
-        <dynamics damping="15" friction="40"/>
+        <dynamics damping="20" friction="50"/>
         <limit lower="-0.55850536063818546" upper="1.5707963267948966" velocity=".17" effort="10000"/>
     </joint>
@@ -264,5 +264,5 @@
       <child link="${namespace}/forearm_axis"/>
       <origin xyz="0.579 0.0 0" rpy="0 1.5707963267948966 0"/>
-      <dynamics damping="15" friction="40"/>
+      <dynamics damping="20" friction="50"/>
       <axis xyz="0 -1 0"/>
       <limit lower="-1.5358897417550099" upper="0.76794487087750496" velocity=".13" effort="10000"/>
@@ -279,5 +279,5 @@
       <origin xyz="0.139 0.0 0" rpy="0 0 0"/>
       <axis xyz="1 0 0"/>
-      <dynamics damping="15" friction="40"/>
+      <dynamics damping="20" friction="50"/>
       <limit lower="-2.3911010752322315" upper="2.3212879051524582" velocity=".085" effort="10000"/>
     </joint>
@@ -287,5 +287,5 @@
       <origin xyz="0.362 0.0 0" rpy="0 0 0"/>
       <axis xyz="0 1 0"/>
-      <dynamics damping="15" friction="40"/>
+      <dynamics damping="20" friction="50"/>
       <limit lower="-1.6406094968746698" upper="0.4537856055185257" velocity=".26" effort="10000"/>
     </joint>

Commit message: CHANGE Damping and friction coefficients for the joints
Signed-off-by: Musa Morena Marcusso Manhães <Musa.Marcusso@de.bosch.com>

File: uuv_manipulators/oberon/oberon_description/urdf/serial_arm.xacro (robot description, xacro)
@@ -249,5 +249,5 @@
       <child link="${namespace}/shoulder_link"/>
       <axis xyz="0 0 1"/>
-      <dynamics damping="20" friction="50"/>
+      <dynamics damping="50" friction="120"/>
       <limit lower="-1.0471975511965976" upper="1.0471975511965976" velocity="0.17" effort="10000"/>
     </joint>
@@ -257,5 +257,5 @@
         <origin xyz="0.07 0.0 0.028" rpy="0 0 0"/>
         <axis xyz="0 -1 0"/>
-        <dynamics damping="20" friction="50"/>
+        <dynamics damping="50" friction="120"/>
         <limit lower="-0.55850536063818546" upper="1.5707963267948966" velocity=".17" effort="10000"/>
     </joint>
@@ -264,5 +264,5 @@
       <child link="${namespace}/forearm_axis"/>
       <origin xyz="0.579 0.0 0" rpy="0 1.5707963267948966 0"/>
-      <dynamics damping="20" friction="50"/>
+      <dynamics damping="50" friction="120"/>
       <axis xyz="0 -1 0"/>
       <limit lower="-1.5358897417550099" upper="0.76794487087750496" velocity=".13" effort="10000"/>
@@ -279,5 +279,5 @@
       <origin xyz="0.139 0.0 0" rpy="0 0 0"/>
       <axis xyz="1 0 0"/>
-      <dynamics damping="20" friction="50"/>
+      <dynamics damping="50" friction="120"/>
       <limit lower="-2.3911010752322315" upper="2.3212879051524582" velocity=".085" effort="10000"/>
     </joint>
@@ -287,5 +287,5 @@
       <origin xyz="0.362 0.0 0" rpy="0 0 0"/>
       <axis xyz="0 1 0"/>
-      <dynamics damping="20" friction="50"/>
+      <dynamics damping="50" friction="120"/>
       <limit lower="-1.6406094968746698" upper="0.4537856055185257" velocity=".26" effort="10000"/>
     </joint>
@@ -295,5 +295,5 @@
       <origin xyz="0.232 0 0" rpy="0 0 0"/>
       <axis xyz="1 0 0"/>
-      <dynamics damping="10" friction="60"/>
+      <dynamics damping="50" friction="120"/>
     </joint>
     <!-- Transmissions -->

Commit message: FIX Name of the link connected to a fixed joint.
Signed-off-by: Musa Morena Marcusso Manhães <Musa.Marcusso@de.bosch.com>

File: uuv_manipulators/oberon/oberon_description/urdf/serial_arm.xacro (robot description, xacro)
@@ -136,9 +136,9 @@
       <selfCollide>false</selfCollide>
     </gazebo>
-    <link name="${namespace}/forearm_axis"/>
-    <gazebo reference="${namespace}/forearm_axis">
-      <selfCollide>false</selfCollide>
-    </gazebo>
-    <link name="${namespace}/forearm">
+    <link name="${namespace}/forearm"/>
+    <gazebo reference="${namespace}/forearm">
+      <selfCollide>false</selfCollide>
+    </gazebo>
+    <link name="${namespace}/forearm_dummy">
       <inertial>
       <origin xyz="0.045 0 -0.043" rpy="0 0 0"/>
@@ -262,5 +262,5 @@
     <joint name="${namespace}/elbow" type="revolute">
       <parent link="${namespace}/upper_arm"/>
-      <child link="${namespace}/forearm_axis"/>
+      <child link="${namespace}/forearm"/>
       <origin xyz="0.579 0.0 0" rpy="0 1.5707963267948966 0"/>
       <dynamics damping="50" friction="120"/>
@@ -269,11 +269,11 @@
     </joint>
     <joint name="${namespace}/elbow_dummy" type="fixed">
-      <parent link="${namespace}/forearm_axis"/>
-      <child link="${namespace}/forearm"/>
+      <parent link="${namespace}/forearm"/>
+      <child link="${namespace}/forearm_dummy"/>
       <origin xyz="0.0 0.0 0.135" rpy="0 0 0"/>
       <axis xyz="1 0 0"/>
     </joint>
     <joint name="${namespace}/roll" type="revolute">
-      <parent link="${namespace}/forearm"/>
+      <parent link="${namespace}/forearm_dummy"/>
       <child link="${namespace}/wrist_1"/>
       <origin xyz="0.139 0.0 0" rpy="0 0 0"/>
