Commit message: ADD Macro for the description of the hydrodynamic models for the manipulator models.
Signed-off-by: Musa Morena Marcusso Manhães <Musa.Marcusso@de.bosch.com>

File: uuv_manipulators/oberon/oberon_description/urdf/serial_arm.gazebo.xacro (robot description, xacro)
@@ -50,76 +50,77 @@
     <implicitSpringDamper>1</implicitSpringDamper>
   </gazebo>
-  <gazebo>
-    <plugin name="uuv_plugin_oberon" filename="libunderwater_object_plugin.so">
-      <fluid_density>1028.0</fluid_density>
-      <flow_velocity_topic>/hydrodynamics/flow_velocity</flow_velocity_topic>
-      <link name="${namespace}/base">
-        <volume>${x1*y1*z1}</volume>
-        <box>
-          <width>${y1}</width>
-          <length>${x1}</length>
-          <height>${z1}</height>
-        </box>
-        <hydrodynamic_model>
-          <type>fossen</type>
-        </hydrodynamic_model>
-      </link>
-      <link name="${namespace}/shoulder_link">
-        <volume>${x2*y2*z2}</volume>
-        <box>
-          <width>${y2}</width>
-          <length>${x2}</length>
-          <height>${z2}</height>
-        </box>
-        <hydrodynamic_model>
-          <type>fossen</type>
-        </hydrodynamic_model>
-      </link>
-      <link name="${namespace}/upper_arm">
-        <volume>${x3*y3*z3}</volume>
-        <box>
-          <width>${y3}</width>
-          <length>${x3}</length>
-          <height>${z3}</height>
-        </box>
-        <hydrodynamic_model>
-          <type>fossen</type>
-        </hydrodynamic_model>
-      </link>
-      <link name="${namespace}/forearm">
-        <volume>${x4*y4*z4}</volume>
-        <box>
-          <width>${y4}</width>
-          <length>${x4}</length>
-          <height>${z4}</height>
-        </box>
-        <hydrodynamic_model>
-          <type>fossen</type>
-        </hydrodynamic_model>
-      </link>
-      <link name="${namespace}/wrist_1">
-        <volume>${x5*y5*z5}</volume>
-        <box>
-          <width>${y5}</width>
-          <length>${x5}</length>
-          <height>${z5}</height>
-        </box>
-        <hydrodynamic_model>
-          <type>fossen</type>
-        </hydrodynamic_model>
-      </link>
-      <link name="${namespace}/wrist_2">
-        <volume>${x6*y6*z6}</volume>
-        <box>
-          <width>${y6}</width>
-          <length>${x6}</length>
-          <height>${z6}</height>
-        </box>
-        <hydrodynamic_model>
-          <type>fossen</type>
-        </hydrodynamic_model>
-      </link>
-    </plugin>
-  </gazebo>
+</xacro:macro>
+<!--
+  Parameters for the uuv_underwater_object_plugin that includes the implementation
+  of Fossen's equations of motion for underwater vehicles. This parameters will
+  be loaded by the vehicle where it is installed.
+-->
+<xacro:macro name="oberon_hydro_model" params="namespace">
+  <link name="${namespace}/base">
+    <volume>${x1*y1*z1}</volume>
+    <box>
+      <width>${y1}</width>
+      <length>${x1}</length>
+      <height>${z1}</height>
+    </box>
+    <hydrodynamic_model>
+      <type>fossen</type>
+    </hydrodynamic_model>
+  </link>
+  <link name="${namespace}/shoulder_link">
+    <volume>${x2*y2*z2}</volume>
+    <box>
+      <width>${y2}</width>
+      <length>${x2}</length>
+      <height>${z2}</height>
+    </box>
+    <hydrodynamic_model>
+      <type>fossen</type>
+    </hydrodynamic_model>
+  </link>
+  <link name="${namespace}/upper_arm">
+    <volume>${x3*y3*z3}</volume>
+    <box>
+      <width>${y3}</width>
+      <length>${x3}</length>
+      <height>${z3}</height>
+    </box>
+    <hydrodynamic_model>
+      <type>fossen</type>
+    </hydrodynamic_model>
+  </link>
+  <link name="${namespace}/forearm">
+    <volume>${x4*y4*z4}</volume>
+    <box>
+      <width>${y4}</width>
+      <length>${x4}</length>
+      <height>${z4}</height>
+    </box>
+    <hydrodynamic_model>
+      <type>fossen</type>
+    </hydrodynamic_model>
+  </link>
+  <link name="${namespace}/wrist_1">
+    <volume>${x5*y5*z5}</volume>
+    <box>
+      <width>${y5}</width>
+      <length>${x5}</length>
+      <height>${z5}</height>
+    </box>
+    <hydrodynamic_model>
+      <type>fossen</type>
+    </hydrodynamic_model>
+  </link>
+  <link name="${namespace}/wrist_2">
+    <volume>${x6*y6*z6}</volume>
+    <box>
+      <width>${y6}</width>
+      <length>${x6}</length>
+      <height>${z6}</height>
+    </box>
+    <hydrodynamic_model>
+      <type>fossen</type>
+    </hydrodynamic_model>
+  </link>
 </xacro:macro>
 </robot>

File: uuv_manipulators/oberon4/oberon4_description/urdf/serial_arm.gazebo.xacro (robot description, xacro)
@@ -56,65 +56,66 @@
     <implicitSpringDamper>1</implicitSpringDamper>
   </gazebo>
-  <gazebo>
-    <plugin name="uuv_plugin_oberon4" filename="libunderwater_object_plugin.so">
-      <fluid_density>1028.0</fluid_density>
-      <flow_velocity_topic>/hydrodynamics/flow_velocity</flow_velocity_topic>
-      <link name="${namespace}/base">
-        <volume>${base_volume}</volume>
-        <box>
-          <width>${base_y}</width>
-          <length>${base_x}</length>
-          <height>${base_z}</height>
-        </box>
-        <hydrodynamic_model>
-          <type>fossen</type>
-        </hydrodynamic_model>
-      </link>
-      <link name="${namespace}/azimuth_link">
-        <volume>${azimuth_volume}</volume>
-        <box>
-          <width>${azimuth_y}</width>
-          <length>${azimuth_x}</length>
-          <height>${azimuth_z}</height>
-        </box>
-        <hydrodynamic_model>
-          <type>fossen</type>
-        </hydrodynamic_model>
-      </link>
-      <link name="${namespace}/arm">
-        <volume>${arm_volume}</volume>
-        <box>
-          <width>${arm_y}</width>
-          <length>${arm_x}</length>
-          <height>${arm_z}</height>
-        </box>
-        <hydrodynamic_model>
-          <type>fossen</type>
-        </hydrodynamic_model>
-      </link>
-      <link name="${namespace}/wrist">
-        <volume>${wrist_volume}</volume>
-        <box>
-          <width>${wrist_y}</width>
-          <length>${wrist_x}</length>
-          <height>${wrist_z}</height>
-        </box>
-        <hydrodynamic_model>
-          <type>fossen</type>
-        </hydrodynamic_model>
-      </link>
-      <link name="${namespace}/gripper_base">
-        <volume>${gripper_base_volume}</volume>
-        <box>
-          <width>${gripper_base_y}</width>
-          <length>${gripper_base_x}</length>
-          <height>${gripper_base_z}</height>
-        </box>
-        <hydrodynamic_model>
-          <type>fossen</type>
-        </hydrodynamic_model>
-      </link>
-    </plugin>
-  </gazebo>
+</xacro:macro>
+<!--
+  Parameters for the uuv_underwater_object_plugin that includes the implementation
+  of Fossen's equations of motion for underwater vehicles. This parameters will
+  be loaded by the vehicle where it is installed.
+-->
+<xacro:macro name="oberon4_hydro_model" params="namespace">
+  <link name="${namespace}/base">
+    <volume>${base_volume}</volume>
+    <box>
+      <width>${base_y}</width>
+      <length>${base_x}</length>
+      <height>${base_z}</height>
+    </box>
+    <hydrodynamic_model>
+      <type>fossen</type>
+    </hydrodynamic_model>
+  </link>
+  <link name="${namespace}/azimuth_link">
+    <volume>${azimuth_volume}</volume>
+    <box>
+      <width>${azimuth_y}</width>
+      <length>${azimuth_x}</length>
+      <height>${azimuth_z}</height>
+    </box>
+    <hydrodynamic_model>
+      <type>fossen</type>
+    </hydrodynamic_model>
+  </link>
+  <link name="${namespace}/arm">
+    <volume>${arm_volume}</volume>
+    <box>
+      <width>${arm_y}</width>
+      <length>${arm_x}</length>
+      <height>${arm_z}</height>
+    </box>
+    <hydrodynamic_model>
+      <type>fossen</type>
+    </hydrodynamic_model>
+  </link>
+  <link name="${namespace}/wrist">
+    <volume>${wrist_volume}</volume>
+    <box>
+      <width>${wrist_y}</width>
+      <length>${wrist_x}</length>
+      <height>${wrist_z}</height>
+    </box>
+    <hydrodynamic_model>
+      <type>fossen</type>
+    </hydrodynamic_model>
+  </link>
+  <link name="${namespace}/gripper_base">
+    <volume>${gripper_base_volume}</volume>
+    <box>
+      <width>${gripper_base_y}</width>
+      <length>${gripper_base_x}</length>
+      <height>${gripper_base_z}</height>
+    </box>
+    <hydrodynamic_model>
+      <type>fossen</type>
+    </hydrodynamic_model>
+  </link>
 </xacro:macro>
 </robot>

Commit message: RM Dummy link and fixed joint from serial arm
Signed-off-by: Musa Morena Marcusso Manhaes <Musa.Marcusso@de.bosch.com>

File: uuv_manipulators/oberon/oberon_description/urdf/serial_arm.gazebo.xacro (robot description, xacro)
@@ -9,7 +9,4 @@
   </gazebo>
   <gazebo reference="${namespace}/upper_arm">
-    <selfCollide>false</selfCollide>
-  </gazebo>
-  <gazebo reference="${namespace}/forearm_axis">
     <selfCollide>false</selfCollide>
   </gazebo>
@@ -36,7 +33,4 @@
   </gazebo>
   <gazebo reference="${namespace}/elbow">
-    <implicitSpringDamper>1</implicitSpringDamper>
-  </gazebo>
-  <gazebo reference="${namespace}/elbow_dummy">
     <implicitSpringDamper>1</implicitSpringDamper>
   </gazebo>

File: uuv_manipulators/oberon/oberon_description/urdf/serial_arm.xacro (robot description, xacro)
@@ -72,7 +72,4 @@
       </collision>
     </link>
-    <gazebo reference="${namespace}/base">
-      <selfCollide>false</selfCollide>
-    </gazebo>
     <link name="${namespace}/shoulder_link">
       <inertial>
@@ -101,7 +98,4 @@
       </collision>
     </link>
-    <gazebo reference="${namespace}/shoulder_link">
-      <selfCollide>false</selfCollide>
-    </gazebo>
     <link name="${namespace}/upper_arm">
       <inertial>
@@ -133,12 +127,5 @@
       </collision>
     </link>
-    <gazebo reference="${namespace}/upper_arm">
-      <selfCollide>false</selfCollide>
-    </gazebo>
-    <link name="${namespace}/forearm"/>
-    <gazebo reference="${namespace}/forearm">
-      <selfCollide>false</selfCollide>
-    </gazebo>
-    <link name="${namespace}/forearm_dummy">
+    <link name="${namespace}/forearm">
       <inertial>
       <origin xyz="0.045 0 -0.043" rpy="0 0 0"/>
@@ -166,7 +153,4 @@
       </collision>
     </link>
-    <gazebo reference="${namespace}/forearm">
-      <selfCollide>false</selfCollide>
-    </gazebo>
     <link name="${namespace}/wrist_1">
       <inertial>
@@ -198,7 +182,4 @@
       </collision>
     </link>
-    <gazebo reference="${namespace}/wrist_1">
-      <selfCollide>false</selfCollide>
-    </gazebo>
     <link name="${namespace}/wrist_2">
       <inertial>
@@ -230,11 +211,5 @@
       </collision>
     </link>
-    <gazebo reference="${namespace}/wrist_2">
-      <selfCollide>false</selfCollide>
-    </gazebo>
     <xacro:dummy_link name="${namespace}/end_effector"/>
-    <gazebo reference="${namespace}/end_effector">
-      <selfCollide>false</selfCollide>
-    </gazebo>
     <!-- All the joints -->
     <joint name="${namespace}/anchor" type="revolute">
@@ -256,26 +231,20 @@
         <child link="${namespace}/upper_arm"/>
         <origin xyz="0.07 0.0 0.028" rpy="0 0 0"/>
-        <axis xyz="0 -1 0"/>
+        <axis xyz="0 1 0"/>
         <dynamics damping="50" friction="120"/>
-        <limit lower="-0.55850536063818546" upper="1.5707963267948966" velocity=".17" effort="10000"/>
+        <limit lower="${-0.5*PI}" upper="${0.5*PI}" velocity=".17" effort="10000"/>
     </joint>
     <joint name="${namespace}/elbow" type="revolute">
       <parent link="${namespace}/upper_arm"/>
       <child link="${namespace}/forearm"/>
-      <origin xyz="0.579 0.0 0" rpy="0 1.5707963267948966 0"/>
+      <origin xyz="0.579 0 0" rpy="0 0 0"/>
       <dynamics damping="50" friction="120"/>
       <axis xyz="0 -1 0"/>
       <limit lower="-1.5358897417550099" upper="0.76794487087750496" velocity=".13" effort="10000"/>
     </joint>
-    <joint name="${namespace}/elbow_dummy" type="fixed">
+    <joint name="${namespace}/roll" type="revolute">
       <parent link="${namespace}/forearm"/>
-      <child link="${namespace}/forearm_dummy"/>
-      <origin xyz="0.0 0.0 0.135" rpy="0 0 0"/>
-      <axis xyz="1 0 0"/>
-    </joint>
-    <joint name="${namespace}/roll" type="revolute">
-      <parent link="${namespace}/forearm_dummy"/>
       <child link="${namespace}/wrist_1"/>
-      <origin xyz="0.139 0.0 0" rpy="0 0 0"/>
+      <origin xyz="0.139 0 -0.14" rpy="0 ${PI*0.5} 0"/>
       <axis xyz="1 0 0"/>
       <dynamics damping="50" friction="120"/>
@@ -286,7 +255,7 @@
       <child link="${namespace}/wrist_2"/>
       <origin xyz="0.362 0.0 0" rpy="0 0 0"/>
-      <axis xyz="0 1 0"/>
-      <dynamics damping="50" friction="120"/>
-      <limit lower="-1.6406094968746698" upper="0.4537856055185257" velocity=".26" effort="10000"/>
+      <axis xyz="0 -1 0"/>
+      <dynamics damping="50" friction="120"/>
+      <limit lower="-0.4537856055185257" upper="1.6406094968746698" velocity=".26" effort="10000"/>
     </joint>
     <joint name="${namespace}/wrist" type="continuous">
