Commit message: Adapting demos for new vehicle teleop.
Signed-off-by: Musa Morena Marcusso Manhães <Musa.Marcusso@de.bosch.com>

File: uuv_manipulators/oberon4/oberon4_description/urdf/serial_arm.xacro (robot description, xacro)
@@ -52,6 +52,17 @@
   <xacro:property name="jaw_z" value="0.091102" />
   <xacro:property name="jaw_center_of_mass" value="0.052693 0.02887 -0.00805"/>
-  <!-- Import common macros-->
-  <xacro:include filename="$(find uuv_manipulators_description)/urdf/common.xacro" />
+  <!-- Transmission Macro -->
+  <xacro:macro name="simple_transmission" params="joint">
+    <transmission name="${joint}_trans">
+      <type>transmission_interface/SimpleTransmission</type>
+      <joint name="${joint}">
+        <hardwareInterface>EffortJointInterface</hardwareInterface>
+      </joint>
+      <actuator name="${joint}_motor">
+        <hardwareInterface>EffortJointInterface</hardwareInterface>
+        <mechanicalReduction>1</mechanicalReduction>
+      </actuator>
+    </transmission>
+  </xacro:macro>
   <!-- Gazebo specific configurations -->
   <xacro:include filename="$(find oberon4_description)/urdf/serial_arm.gazebo.xacro" />

Commit message: Adjusting gripper joint dynamics.
Signed-off-by: Musa Morena Marcusso Manhães <Musa.Marcusso@de.bosch.com>

File: uuv_manipulators/oberon4/oberon4_description/urdf/serial_arm.xacro (robot description, xacro)
@@ -273,5 +273,5 @@
       <child link="${namespace}/jaw_2"/>
       <origin xyz="0.0444253 -0.021926 -0.0487509" rpy="${0.5*PI} 0 0"/>
-      <dynamics damping="15" friction="10"/>
+      <dynamics damping="5" friction="10"/>
       <axis xyz="0 0 1"/>
       <limit lower="${-0.5*PI}" upper="0" velocity=".13" effort="50000"/>

Commit message: Corrections to improve stability.
Signed-off-by: Musa Morena Marcusso Manhães <Musa.Marcusso@de.bosch.com>

File: uuv_manipulators/oberon4/oberon4_description/urdf/serial_arm.xacro (robot description, xacro)
@@ -266,5 +266,5 @@
       <dynamics damping="15" friction="10"/>
       <axis xyz="0 0 1"/>
-      <limit lower="${-0.5*PI}" upper="0" velocity=".13" effort="50000"/>
+      <limit lower="${-0.5*PI}" upper="0" velocity=".1" effort="100"/>
       <mimic joint="${namespace}/jaw_1_joint"/>
     </joint>
@@ -275,5 +275,5 @@
       <dynamics damping="5" friction="10"/>
       <axis xyz="0 0 1"/>
-      <limit lower="${-0.5*PI}" upper="0" velocity=".13" effort="50000"/>
+      <limit lower="${-0.5*PI}" upper="0" velocity=".1" effort="100"/>
     </joint>
     <!-- Transmissions -->
