Commit message: add axis to gps joint as required by kdl_parser.py
Signed-off-by: Sebastian Scherer <sebastian.scherer2@de.bosch.com>

File: uuv_sensor_plugins/uuv_sensor_plugins_ros/urdf/gps_sensor_snippets.xacro (robot description, xacro)
@@ -30,4 +30,5 @@
       <parent link="${parent_link}" />
       <child link="${namespace}/gps_link" />
+      <axis xyz="1 0 0"/>
       <limit upper="0" lower="0" effort="0" velocity="0" />
     </joint>
