Commit message: Add optical frame to camera.
Signed-off-by: Luiz Ricardo Douat <luizricardo.douat@de.bosch.com>

File: uuv_sensor_plugins/uuv_sensor_plugins_ros/urdf/camera_snippets.xacro (robot description, xacro)
@@ -78,4 +78,24 @@
     <parent link="${parent_link}" />
     <child link="${namespace}/camera${suffix}_link" />
+    <limit upper="0" lower="0" effort="0" velocity="0" />
+    <axis xyz="1 0 0"/>
+  </joint>
+  <link name="${namespace}/camera${suffix}_link_optical">
+    <xacro:box_inertial x="0" y="0" z="0" mass="0.001">
+      <origin xyz="0 0 0" rpy="0 0 0"/>
+    </xacro:box_inertial>
+    <collision>
+      <!-- todo: gazebo needs a collision volume or it will ignore the pose of
+         the joint that leads to this link (and assume it to be the identity) -->
+      <geometry>
+        <cylinder length="0.000001" radius="0.000001"/>
+      </geometry>
+      <origin xyz="0 0 0" rpy="0 ${0.5*pi} 0"/>
+    </collision>
+  </link>
+  <joint name="${namespace}/camera${suffix}_optical_joint" type="revolute">
+    <origin xyz="0 0 0" rpy="${-pi/2} 0 ${-pi/2}"/>
+    <parent link="${namespace}/camera${suffix}_link"/>
+    <child link="${namespace}/camera${suffix}_link_optical"/>
     <limit upper="0" lower="0" effort="0" velocity="0" />
     <axis xyz="1 0 0"/>
@@ -104,5 +124,5 @@
         <updateRate>${update_rate}</updateRate>
         <cameraName>${namespace}/camera${suffix}</cameraName>
-        <frameName>${namespace}/camera${suffix}_link</frameName>
+        <frameName>camera${suffix}_link_optical</frameName>
         <attenuationR>0.0</attenuationR>
         <attenuationG>0.0</attenuationG>

Commit message: FIX Null inertial in the camera optical link
Signed-off-by: Musa Morena Marcusso Manhaes <Musa.Marcusso@de.bosch.com>

File: uuv_sensor_plugins/uuv_sensor_plugins_ros/urdf/camera_snippets.xacro (robot description, xacro)
@@ -28,5 +28,5 @@
       parent_link="${parent_link}"
       topic="camera"
-      mass="0.001"
+      mass="0.1"
       update_rate="30"
       hfov="1.5125"
@@ -36,5 +36,5 @@
       scale="1.0">
       <inertia ixx="0.00001" ixy="0.0" ixz="0.0" iyy="0.00001" iyz="0.0" izz="0.00001" />
-      <xacro:insert_block name="origin" />>
+      <xacro:insert_block name="origin" />
     </xacro:regular_camera_plugin_macro>
   </xacro:macro>
@@ -82,5 +82,5 @@
   </joint>
   <link name="${namespace}/camera${suffix}_link_optical">
-    <xacro:box_inertial x="0" y="0" z="0" mass="0.001">
+    <xacro:box_inertial x="0.0001" y="0.0001" z="0.0001" mass="0.001">
       <origin xyz="0 0 0" rpy="0 0 0"/>
     </xacro:box_inertial>
@@ -163,4 +163,5 @@
     <parent link="${parent_link}" />
     <child link="${namespace}/camera${suffix}_link" />
+    <axis xyz="1 0 0"/>
     <limit upper="0" lower="0" effort="0" velocity="0" />
   </joint>

Commit message: ADD URDF snippets to Gazebo ROS plugins
Signed-off-by: Musa Morena Marcusso Manhaes <Musa.Marcusso@de.bosch.com>

File: uuv_sensor_plugins/uuv_sensor_plugins_ros/urdf/camera_snippets.xacro (robot description, xacro)
@@ -74,70 +74,70 @@
       <xacro:no_collision/>
     </link>
-  <joint name="${namespace}/camera${suffix}_joint" type="revolute">
-    <xacro:insert_block name="origin" />
-    <parent link="${parent_link}" />
-    <child link="${namespace}/camera${suffix}_link" />
-    <limit upper="0" lower="0" effort="0" velocity="0" />
-    <axis xyz="1 0 0"/>
-  </joint>
-  <link name="${namespace}/camera${suffix}_link_optical">
-    <xacro:box_inertial x="0.0001" y="0.0001" z="0.0001" mass="0.001">
-      <origin xyz="0 0 0" rpy="0 0 0"/>
-    </xacro:box_inertial>
-    <collision>
-      <!-- todo: gazebo needs a collision volume or it will ignore the pose of
-         the joint that leads to this link (and assume it to be the identity) -->
-      <geometry>
-        <cylinder length="0.000001" radius="0.000001"/>
-      </geometry>
-      <origin xyz="0 0 0" rpy="0 ${0.5*pi} 0"/>
-    </collision>
-  </link>
-  <joint name="${namespace}/camera${suffix}_optical_joint" type="revolute">
-    <origin xyz="0 0 0" rpy="${-pi/2} 0 ${-pi/2}"/>
-    <parent link="${namespace}/camera${suffix}_link"/>
-    <child link="${namespace}/camera${suffix}_link_optical"/>
-    <limit upper="0" lower="0" effort="0" velocity="0" />
-    <axis xyz="1 0 0"/>
-  </joint>
-  <gazebo reference="${namespace}/camera${suffix}_link">
-    <sensor type="camera" name="camera${suffix}">
-      <update_rate>${update_rate}</update_rate>
-      <camera name="camera${suffix}">
-        <horizontal_fov>${hfov}</horizontal_fov>
-        <image>
-          <width>${width}</width>
-          <height>${height}</height>
-          <format>R8G8B8</format>
-        </image>
-        <clip>
-          <near>0.05</near>
-          <far>3000</far>
-        </clip>
-        <noise>
-          <type>gaussian</type>
-          <mean>0.0</mean>
-          <stddev>${stddev}</stddev>
-        </noise>
-      </camera>
-      <plugin name="camera${suffix}_controller" filename="libgazebo_ros_camera.so">
-        <updateRate>${update_rate}</updateRate>
-        <cameraName>${namespace}/camera${suffix}</cameraName>
-        <frameName>camera${suffix}_link_optical</frameName>
-        <attenuationR>0.0</attenuationR>
-        <attenuationG>0.0</attenuationG>
-        <attenuationB>0.0</attenuationB>
-        <backgroundR>0</backgroundR>
-        <backgroundG>0</backgroundG>
-        <backgroundB>0</backgroundB>
-        <!-- required for ros depth cam -->
-        <imageTopicName>${topic}_image</imageTopicName>
-        <pointCloudTopicName>${topic}_cloud</pointCloudTopicName>
-        <depthImageTopicName>${topic}_depth</depthImageTopicName>
-        <depthImageCameraInfoTopicName>${topic}_depth_info</depthImageCameraInfoTopicName>
-        <pointCloudCutoff>10.0</pointCloudCutoff>
-      </plugin>
-    </sensor>
-  </gazebo>
+    <joint name="${namespace}/camera${suffix}_joint" type="revolute">
+      <xacro:insert_block name="origin" />
+      <parent link="${parent_link}" />
+      <child link="${namespace}/camera${suffix}_link" />
+      <limit upper="0" lower="0" effort="0" velocity="0" />
+      <axis xyz="1 0 0"/>
+    </joint>
+    <link name="${namespace}/camera${suffix}_link_optical">
+      <xacro:box_inertial x="0.0001" y="0.0001" z="0.0001" mass="0.001">
+        <origin xyz="0 0 0" rpy="0 0 0"/>
+      </xacro:box_inertial>
+      <collision>
+        <!-- todo: gazebo needs a collision volume or it will ignore the pose of
+           the joint that leads to this link (and assume it to be the identity) -->
+        <geometry>
+          <cylinder length="0.000001" radius="0.000001"/>
+        </geometry>
+        <origin xyz="0 0 0" rpy="0 ${0.5*pi} 0"/>
+      </collision>
+    </link>
+    <joint name="${namespace}/camera${suffix}_optical_joint" type="revolute">
+      <origin xyz="0 0 0" rpy="${-pi/2} 0 ${-pi/2}"/>
+      <parent link="${namespace}/camera${suffix}_link"/>
+      <child link="${namespace}/camera${suffix}_link_optical"/>
+      <limit upper="0" lower="0" effort="0" velocity="0" />
+      <axis xyz="1 0 0"/>
+    </joint>
+    <gazebo reference="${namespace}/camera${suffix}_link">
+      <sensor type="camera" name="camera${suffix}">
+        <update_rate>${update_rate}</update_rate>
+        <camera name="camera${suffix}">
+          <horizontal_fov>${hfov}</horizontal_fov>
+          <image>
+            <width>${width}</width>
+            <height>${height}</height>
+            <format>R8G8B8</format>
+          </image>
+          <clip>
+            <near>0.05</near>
+            <far>3000</far>
+          </clip>
+          <noise>
+            <type>gaussian</type>
+            <mean>0.0</mean>
+            <stddev>${stddev}</stddev>
+          </noise>
+        </camera>
+        <plugin name="camera${suffix}_controller" filename="libgazebo_ros_camera.so">
+          <updateRate>${update_rate}</updateRate>
+          <cameraName>${namespace}/camera${suffix}</cameraName>
+          <frameName>camera${suffix}_link_optical</frameName>
+          <attenuationR>0.0</attenuationR>
+          <attenuationG>0.0</attenuationG>
+          <attenuationB>0.0</attenuationB>
+          <backgroundR>0</backgroundR>
+          <backgroundG>0</backgroundG>
+          <backgroundB>0</backgroundB>
+          <!-- required for ros depth cam -->
+          <imageTopicName>${topic}_image</imageTopicName>
+          <pointCloudTopicName>${topic}_cloud</pointCloudTopicName>
+          <depthImageTopicName>${topic}_depth</depthImageTopicName>
+          <depthImageCameraInfoTopicName>${topic}_depth_info</depthImageCameraInfoTopicName>
+          <pointCloudCutoff>10.0</pointCloudCutoff>
+        </plugin>
+      </sensor>
+    </gazebo>
   </xacro:macro>
   <xacro:macro name="underwater_camera_plugin_macro"
@@ -159,50 +159,50 @@
       <xacro:no_collision/>
     </link>
-  <joint name="${namespace}/camera${suffix}_joint" type="revolute">
-    <xacro:insert_block name="origin" />
-    <parent link="${parent_link}" />
-    <child link="${namespace}/camera${suffix}_link" />
-    <axis xyz="1 0 0"/>
-    <limit upper="0" lower="0" effort="0" velocity="0" />
-  </joint>
-  <gazebo reference="${namespace}/camera${suffix}_link">
-    <sensor type="depth" name="camera${suffix}">
-      <update_rate>${update_rate}</update_rate>
-      <camera name="camera${suffix}">
-        <horizontal_fov>${hfov}</horizontal_fov>
-        <image>
-          <width>${width}</width>
-          <height>${height}</height>
-          <format>R8G8B8</format>
-        </image>
-        <clip>
-          <near>0.1</near>
-          <far>3000</far>
-        </clip>
-        <noise>
-          <type>gaussian</type>
-          <mean>0.0</mean>
-          <stddev>${stddev}</stddev>
-        </noise>
-      </camera>
-      <plugin name="camera${suffix}_controller" filename="libuuv_gazebo_ros_camera.so">
-        <updateRate>${update_rate}</updateRate>
-        <cameraName>${namespace}/camera${suffix}</cameraName>
-        <frameName>${namespace}/camera${suffix}_link</frameName>
-        <attenuationR>0.01</attenuationR>
-        <attenuationG>0.01</attenuationG>
-        <attenuationB>0.003</attenuationB>
-        <backgroundR>0</backgroundR>
-        <backgroundG>0</backgroundG>
-        <backgroundB>0</backgroundB>
-        <!-- required for ros depth cam -->
-        <imageTopicName>${topic}_image</imageTopicName>
-        <pointCloudTopicName>${topic}_cloud</pointCloudTopicName>
-        <depthImageTopicName>${topic}_depth</depthImageTopicName>
-        <depthImageCameraInfoTopicName>${topic}_depth_info</depthImageCameraInfoTopicName>
-        <pointCloudCutoff>10.0</pointCloudCutoff>
-      </plugin>
-    </sensor>
-  </gazebo>
+    <joint name="${namespace}/camera${suffix}_joint" type="revolute">
+      <xacro:insert_block name="origin" />
+      <parent link="${parent_link}" />
+      <child link="${namespace}/camera${suffix}_link" />
+      <axis xyz="1 0 0"/>
+      <limit upper="0" lower="0" effort="0" velocity="0" />
+    </joint>
+    <gazebo reference="${namespace}/camera${suffix}_link">
+      <sensor type="depth" name="camera${suffix}">
+        <update_rate>${update_rate}</update_rate>
+        <camera name="camera${suffix}">
+          <horizontal_fov>${hfov}</horizontal_fov>
+          <image>
+            <width>${width}</width>
+            <height>${height}</height>
+            <format>R8G8B8</format>
+          </image>
+          <clip>
+            <near>0.1</near>
+            <far>3000</far>
+          </clip>
+          <noise>
+            <type>gaussian</type>
+            <mean>0.0</mean>
+            <stddev>${stddev}</stddev>
+          </noise>
+        </camera>
+        <plugin name="camera${suffix}_controller" filename="libuuv_gazebo_ros_camera.so">
+          <updateRate>${update_rate}</updateRate>
+          <cameraName>${namespace}/camera${suffix}</cameraName>
+          <frameName>${namespace}/camera${suffix}_link</frameName>
+          <attenuationR>0.01</attenuationR>
+          <attenuationG>0.01</attenuationG>
+          <attenuationB>0.003</attenuationB>
+          <backgroundR>0</backgroundR>
+          <backgroundG>0</backgroundG>
+          <backgroundB>0</backgroundB>
+          <!-- required for ros depth cam -->
+          <imageTopicName>${topic}_image</imageTopicName>
+          <pointCloudTopicName>${topic}_cloud</pointCloudTopicName>
+          <depthImageTopicName>${topic}_depth</depthImageTopicName>
+          <depthImageCameraInfoTopicName>${topic}_depth_info</depthImageCameraInfoTopicName>
+          <pointCloudCutoff>10.0</pointCloudCutoff>
+        </plugin>
+      </sensor>
+    </gazebo>
   </xacro:macro>
 </robot>
