Commit message: CHANGE Gazebo SDF description
Signed-off-by: Musa Morena Marcusso Manhaes <Musa.Marcusso@de.bosch.com>

File: uuv_manipulators/oberon7/oberon7_description/models/oberon7/model.urdf (robot description, URDF)
Before this commit: robot oberon7, 12 links, 11 joints
Joints:
- joint /finger_left_joint: origin xyz=0 0.0391376 0.0444267 rpy=0 -1.57079632679 0 -> xyz=0.0444267 0.0391376 0 rpy=0 0 0
- joint /finger_right_joint: limit lower=-1.04709283144 upper=0 effort=30 velocity=0.15 -> lower=0 upper=1.04709283144 effort=30 velocity=0.15; origin xyz=0 -0.0391376 0.0444267 rpy=3.14159265359 -1.57079632679 3.14159265359 -> xyz=0.0444267 -0.0391376 0 rpy=3.14159265359 3.14159265359 3.14159265359
- joint /wrist: axis 0 0 1 -> 1 0 0; origin xyz=0.19304 0 0 rpy=0 1.57079632679 0 -> xyz=0.19304 0 0 rpy=0 0 0

Commit message: CHANGE Simplification of the collision geometries.
Signed-off-by: Musa Morena Marcusso Manhaes <Musa.Marcusso@de.bosch.com>

File: uuv_manipulators/oberon7/oberon7_description/models/oberon7/model.urdf (robot description, URDF)
Before this commit: robot oberon7, 12 links, 11 joints
Links:
- link /elbow_link: geometry collision cylinder length=0.245312 radius=0.077562; visual mesh filename=file:///home/mam0box/catkin_ws/src/uuv_simulator/uuv_manipu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
- link /end_effector: geometry collision box size=0.074326 0.117427 0.114298; visual mesh filename=file:///home/mam0box/catkin_ws/src/uuv_simulator/uuv_manipu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
- link /forearm: geometry collision cylinder length=0.334827 radius=0.0757275; visual mesh filename=file:///home/mam0box/catkin_ws/src/uuv_simulator/uuv_manipu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
- link /shoulder_link: geometry collision cylinder length=0.239627 radius=0.068184; visual mesh filename=file:///home/mam0box/catkin_ws/src/uuv_simulator/uuv_manipu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
- link /upper_arm: geometry collision cylinder length=0.616809 radius=0.0709445; visual mesh filename=file:///home/mam0box/catkin_ws/src/uuv_simulator/uuv_manipu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
- link /wrist_link: geometry collision cylinder length=0.219204 radius=0.065187; visual mesh filename=file:///home/mam0box/catkin_ws/src/uuv_simulator/uuv_manipu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
Joints:
- joint /elbow: limit lower=-1.57079637 upper=1.04719758 effort=200 velocity=.13 -> lower=-1.57079637 upper=1.04719758 effort=300 velocity=.13

File: uuv_manipulators/oberon7/oberon7_description/urdf/parallel_gripper.xacro (robot description, xacro)
@@ -28,7 +28,7 @@
         </visual>
         <collision>
-            <origin xyz="0 0 0" rpy="0 0 0"/>
+            <origin xyz="${gripper_base_com}" rpy="0 0 0"/>
             <geometry>
-                <mesh filename="file://$(find oberon7_description)/meshes/parallel_gripper/visual/BaseGripper.dae"/>
+                <box size="${gripper_base_length} ${gripper_base_width} ${gripper_base_height}"/>
             </geometry>
         </collision>

File: uuv_manipulators/oberon7/oberon7_description/urdf/parameters/parallel_gripper.xacro (robot description, xacro)
@@ -17,26 +17,16 @@
   <!--
     GRIPPER BASE
-    Mesh Bounding Box Size 0.117427 0.114298 0.074326
+    Mesh Bounding Box Size 0.074326 0.117427 0.114298
     Mesh Bounding Box Diag 0.179938
     Mesh Volume is 0.000699
     Mesh Surface is 0.160112
-    Thin shell barycenter 0.000000 0.000018 0.025369
-    Center of Mass is 0.000000 0.000014 0.024426
-    Inertia Tensor is :
-    | 0.000001 -0.000000 0.000000 |
-    | -0.000000 0.000001 -0.000000 |
-    | 0.000000 -0.000000 0.000001 |
-    Principal axes are :
-    | 1.000000 -0.000000 0.000001 |
-    | 0.000000 1.000000 -0.000842 |
-    | -0.000001 0.000842 1.000000 |
-    axis momenta are :
-    | 0.000001 0.000001 0.000001 |
+    Thin shell barycenter 0.025369 -0.000000 -0.000018
+    Center of Mass is 0.024426 -0.000000 -0.000014
   -->
   <xacro:property name="gripper_base_width" value="0.117427" />
-  <xacro:property name="gripper_base_length" value="0.114298" />
-  <xacro:property name="gripper_base_height" value="0.074326" />
+  <xacro:property name="gripper_base_length" value="0.074326" />
+  <xacro:property name="gripper_base_height" value="0.114298" />
   <xacro:property name="gripper_base_volume" value="${gripper_base_width * gripper_base_length * gripper_base_height}"/>
-  <xacro:property name="gripper_base_com" value="0.000000 0.000014 0.024426" />
+  <xacro:property name="gripper_base_com" value="0.024426 -0.000000 -0.000014" />
   <!--
     FINGER
@@ -47,14 +37,4 @@
     Thin shell barycenter 0.030139 -0.002041 -0.000073
     Center of Mass is 0.025268 -0.001931 -0.000079
-    Inertia Tensor is :
-    | 0.000000 -0.000000 -0.000000 |
-    | -0.000000 0.000000 -0.000000 |
-    | -0.000000 -0.000000 0.000000 |
-    Principal axes are :
-    | 0.992844 -0.119416 -0.000723 |
-    | 0.119417 0.992843 0.001760 |
-    | 0.000507 -0.001834 0.999998 |
-    axis momenta are :
-    | 0.000000 0.000000 0.000000 |
   -->
   <xacro:property name="finger_width" value="0.052970" />
@@ -71,14 +51,4 @@
     Thin shell barycenter 0.025479 0.015748 -0.000000
     Center of Mass is 0.027744 0.017278 -0.000000
-    Inertia Tensor is :
-    | 0.000000 -0.000000 -0.000000 |
-    | -0.000000 0.000000 0.000000 |
-    | -0.000000 0.000000 0.000000 |
-    Principal axes are :
-    | 0.933245 -0.359241 -0.000000 |
-    | 0.359241 0.933245 -0.000000 |
-    | 0.000000 0.000000 1.000000 |
-    axis momenta are :
-    | 0.000000 0.000000 0.000000 |
   -->
   <xacro:property name="finger_tip_width" value="0.050457" />

File: uuv_manipulators/oberon7/oberon7_description/urdf/serial_arm.xacro (robot description, xacro)
@@ -65,7 +65,7 @@
             </visual>
             <collision>
-                <origin xyz="0 0 0" rpy="0 0 0"/>
-                <geometry>
-                    <mesh filename="file://$(find oberon7_description)/meshes/serial_arm/visual/ShoulderLink.dae"/>
+                <origin xyz="${shoulder_link_com}" rpy="0 0 0"/>
+                <geometry>
+                    <cylinder radius="${0.5 * shoulder_link_width}" length="${shoulder_link_height}" />
                 </geometry>
             </collision>
@@ -94,7 +94,7 @@
             </visual>
             <collision>
-                <origin xyz="0 0 0" rpy="0 0 0"/>
-                <geometry>
-                    <mesh filename="file://$(find oberon7_description)/meshes/serial_arm/visual/UpperArm.dae"/>
+                <origin xyz="${upper_arm_com}" rpy="0 ${0.5*pi} 0"/>
+                <geometry>
+                    <cylinder radius="${0.5 * upper_arm_width}" length="${upper_arm_length}"/>
                 </geometry>
             </collision>
@@ -103,5 +103,5 @@
             <parent link="${namespace}/shoulder_link"/>
             <child link="${namespace}/upper_arm"/>
-            <origin xyz="0.06955 0.00015 0.01536" rpy="${0.5*PI} 0 0"/>
+            <origin xyz="0.06955 0.00015 0.01536" rpy="${0.5*pi} 0 0"/>
             <axis xyz="0 0 1"/>
             <dynamics damping="50" friction="120"/>
@@ -124,7 +124,7 @@
             </visual>
             <collision>
-                <origin xyz="0 0 0" rpy="0 0 0"/>
-                <geometry>
-                    <mesh filename="file://$(find oberon7_description)/meshes/serial_arm/visual/ElbowLink.dae"/>
+                <origin xyz="${elbow_link_com}" rpy="0 ${0.5*pi} ${0.5*pi}"/>
+                <geometry>
+                    <cylinder radius="${0.5 * elbow_link_height}" length="${elbow_link_length}"/>
                 </geometry>
             </collision>
@@ -154,7 +154,7 @@
             </visual>
             <collision>
-                <origin xyz="0 0 0" rpy="0 0 0"/>
-                <geometry>
-                    <mesh filename="file://$(find oberon7_description)/meshes/serial_arm/visual/Forearm.dae"/>
+                <origin xyz="${forearm_com}" rpy="0 0 0"/>
+                <geometry>
+                    <cylinder radius="${0.5 * forearm_width}" length="${forearm_height}"/>
                 </geometry>
             </collision>
@@ -184,7 +184,7 @@
             </visual>
             <collision>
-                <origin xyz="0 0 0" rpy="0 0 0"/>
-                <geometry>
-                    <mesh filename="file://$(find oberon7_description)/meshes/serial_arm/visual/Wrist.dae"/>
+                <origin xyz="${wrist_com}" rpy="0 ${0.5*pi} 0"/>
+                <geometry>
+                    <cylinder radius="${0.5 * wrist_height}" length="${wrist_length}"/>
                 </geometry>
             </collision>
