Commit message: FIX Orientation of the end-effector frame.
Signed-off-by: Musa Morena Marcusso Manhaes <Musa.Marcusso@de.bosch.com>

File: uuv_manipulators/oberon7/oberon7_description/urdf/parallel_gripper.xacro (robot description, xacro)
@@ -37,6 +37,6 @@
       <parent link="${namespace}/wrist_link"/>
       <child link="${namespace}/end_effector"/>
-       <origin xyz="0.19304 0 0" rpy="0 ${0.5 * PI} 0"/>
-      <axis xyz="0 0 1"/>
+       <origin xyz="0.19304 0 0" rpy="0 0 0"/>
+      <axis xyz="1 0 0"/>
       <dynamics damping="10" friction="5"/>
     </joint>
@@ -66,5 +66,5 @@
         <parent link="${namespace}/end_effector"/>
         <child link="${namespace}/finger_left"/>
-        <origin xyz="0 0.0391376 0.0444267" rpy="0 ${-0.5 * PI} 0"/>
+        <origin xyz="0.0444267 0.0391376 0" rpy="0 0 0"/>
         <axis xyz="0 0 1"/>
         <dynamics damping="5" friction="10"/>
@@ -125,5 +125,5 @@
         <parent link="${namespace}/end_effector"/>
         <child link="${namespace}/finger_right"/>
-        <origin xyz="0 -0.0391376 0.0444267" rpy="${PI} ${-0.5 * PI} ${PI}"/>
+        <origin xyz="0.0444267 -0.0391376 0" rpy="${PI} ${PI} ${PI}"/>
         <axis xyz="0 0 -1"/>
         <dynamics damping="5" friction="10"/>

File: uuv_manipulators/oberon7/oberon7_description/urdf/serial_arm.xacro (robot description, xacro)
@@ -46,5 +46,5 @@
                 <origin xyz="0 0 0" rpy="0 0 0"/>
                 <geometry>
-                    <mesh filename="file://$(find oberon7_description)/meshes/serial_arm/visual/Base.dae"/>
+                    <mesh filename="file://$(find oberon7_description)/meshes/serial_arm/collision/Base.stl"/>
                 </geometry>
             </collision>
@@ -136,5 +136,5 @@
             <dynamics damping="50" friction="120"/>
             <axis xyz="0 0 1"/>
-            <limit lower="${-90 * d2r}" upper="${60 * d2r}" velocity=".13" effort="200"/>
+            <limit lower="${-90 * d2r}" upper="${60 * d2r}" velocity=".13" effort="300"/>
         </joint>
         <xacro:simple_transmission joint="${namespace}/elbow" />

Commit message: FIX Joint dynamics parameters for Oberon7
Signed-off-by: Musa Morena Marcusso Manhaes <Musa.Marcusso@de.bosch.com>

File: uuv_manipulators/oberon7/oberon7_description/urdf/parallel_gripper.xacro (robot description, xacro)
@@ -34,10 +34,11 @@
         </collision>
     </link>
-    <joint name="${namespace}/wrist" type="continuous">
+    <joint name="${namespace}/wrist" type="revolute">
       <parent link="${namespace}/wrist_link"/>
       <child link="${namespace}/end_effector"/>
-       <origin xyz="0.19304 0 0" rpy="0 0 0"/>
+       <origin xyz="0.19304 0 0" rpy="${-PI*0.5} 0 0"/>
       <axis xyz="1 0 0"/>
       <dynamics damping="10" friction="5"/>
+      <limit effort="10" lower="${-2*PI}" upper="${2*PI}" velocity="${gripper_velocity}"/>
     </joint>
     <xacro:simple_transmission joint="${namespace}/wrist" />

File: uuv_manipulators/oberon7/oberon7_description/urdf/serial_arm.xacro (robot description, xacro)
@@ -16,5 +16,5 @@
     <xacro:include filename="$(find oberon7_description)/urdf/parameters/serial_arm.xacro" />
     <!-- Transmission Macro -->
-    <xacro:macro name="simple_transmission" params="joint">
+    <!-- <xacro:macro name="simple_transmission" params="joint">
         <transmission name="${joint}_trans">
             <type>transmission_interface/SimpleTransmission</type>
@@ -27,4 +27,17 @@
             </actuator>
         </transmission>
+    </xacro:macro> -->
+    <!-- Transmission Macro -->
+    <xacro:macro name="simple_transmission" params="joint">
+      <transmission name="${joint}_trans">
+        <type>transmission_interface/SimpleTransmission</type>
+        <joint name="${joint}">
+          <hardwareInterface>EffortJointInterface</hardwareInterface>
+        </joint>
+        <actuator name="${joint}_motor">
+          <hardwareInterface>EffortJointInterface</hardwareInterface>
+          <mechanicalReduction>1</mechanicalReduction>
+        </actuator>
+      </transmission>
     </xacro:macro>
     <xacro:macro name="oberon7_serial_arm" params="namespace">
@@ -75,6 +88,7 @@
             <child link="${namespace}/shoulder_link"/>
             <axis xyz="0 0 1"/>
-            <dynamics damping="50" friction="120"/>
+            <dynamics damping="50" friction="200"/>
             <limit lower="${-60 * d2r}" upper="${60 * d2r}" velocity="0.17" effort="200"/>
+            <!-- <limit lower="${-60 * d2r}" upper="${60 * d2r}" velocity="0.17" effort="1000"/> -->
         </joint>
         <xacro:simple_transmission joint="${namespace}/azimuth" />
@@ -105,6 +119,7 @@
             <origin xyz="0.06955 0.00015 0.01536" rpy="${0.5*pi} 0 0"/>
             <axis xyz="0 0 1"/>
-            <dynamics damping="50" friction="120"/>
+            <dynamics damping="50" friction="200"/>
             <limit lower="${-90 * d2r}" upper="${90 * d2r}" velocity=".17" effort="5000"/>
+            <!-- <limit lower="${-90 * d2r}" upper="${90 * d2r}" velocity=".17" effort="1000"/> -->
         </joint>
         <xacro:simple_transmission joint="${namespace}/shoulder" />
@@ -134,7 +149,8 @@
             <child link="${namespace}/elbow_link"/>
             <origin xyz="0.55616 -0.01229 0" rpy="0 0 0"/>
-            <dynamics damping="50" friction="120"/>
-            <axis xyz="0 0 1"/>
-            <limit lower="${-90 * d2r}" upper="${60 * d2r}" velocity=".13" effort="1000"/>
+            <dynamics damping="50" friction="200"/>
+            <axis xyz="0 0 1"/>
+            <limit lower="${-90 * d2r}" upper="${60 * d2r}" velocity=".15" effort="300"/>
+            <!-- <limit lower="${-90 * d2r}" upper="${60 * d2r}" velocity=".13" effort="1000"/> -->
         </joint>
         <xacro:simple_transmission joint="${namespace}/elbow" />
@@ -165,6 +181,7 @@
             <origin xyz="0.1349014 -0.1936267 0" rpy="${0.5*PI} 0 0"/>
             <axis xyz="0 0 1"/>
-            <dynamics damping="50" friction="120"/>
-            <limit lower="${-135 * d2r}" upper="${135 * d2r}" velocity=".085" effort="1000"/>
+            <dynamics damping="50" friction="200"/>
+            <!-- <limit lower="${-135 * d2r}" upper="${135 * d2r}" velocity=".15" effort="200"/> -->
+            <limit lower="${-135 * d2r}" upper="${135 * d2r}" velocity=".25" effort="1000"/>
         </joint>
         <xacro:simple_transmission joint="${namespace}/roll" />
@@ -195,6 +212,7 @@
             <origin xyz="0 0 0.31595760629823427" rpy="${-0.5*PI} ${-0.5*PI} 0"/>
             <axis xyz="0 0 1"/>
-            <dynamics damping="50" friction="120"/>
-            <limit lower="${-90 * d2r}" upper="${90 * d2r}" velocity=".26" effort="1000"/>
+            <dynamics damping="50" friction="200"/>
+            <limit lower="${-90 * d2r}" upper="${90 * d2r}" velocity=".26" effort="200"/>
+            <!-- <limit lower="${-90 * d2r}" upper="${90 * d2r}" velocity=".26" effort="1000"/> -->
         </joint>
         <xacro:simple_transmission joint="${namespace}/pitch" />
