Commit message: FIX: Change manipulator Jacobian Transpose controller configuration parameters in order to cope with semi-autonomous manipulation
Signed-off-by: Luiz Ricardo Douat <luizricardo.douat@de.bosch.com>

File: uuv_manipulators/oberon7/oberon7_description/urdf/serial_arm.xacro (robot description, xacro)
@@ -88,7 +88,6 @@
             <child link="${namespace}/shoulder_link"/>
             <axis xyz="0 0 1"/>
-            <dynamics damping="50" friction="200"/>
+            <dynamics damping="100" friction="150"/>
             <limit lower="${-60 * d2r}" upper="${60 * d2r}" velocity="0.17" effort="200"/>
-            <!-- <limit lower="${-60 * d2r}" upper="${60 * d2r}" velocity="0.17" effort="1000"/> -->
         </joint>
         <xacro:simple_transmission joint="${namespace}/azimuth" />
@@ -119,7 +118,6 @@
             <origin xyz="0.06955 0.00015 0.01536" rpy="${0.5*pi} 0 0"/>
             <axis xyz="0 0 1"/>
-            <dynamics damping="50" friction="200"/>
+            <dynamics damping="50" friction="150"/>
             <limit lower="${-90 * d2r}" upper="${90 * d2r}" velocity=".17" effort="5000"/>
-            <!-- <limit lower="${-90 * d2r}" upper="${90 * d2r}" velocity=".17" effort="1000"/> -->
         </joint>
         <xacro:simple_transmission joint="${namespace}/shoulder" />
@@ -149,8 +147,7 @@
             <child link="${namespace}/elbow_link"/>
             <origin xyz="0.55616 -0.01229 0" rpy="0 0 0"/>
-            <dynamics damping="50" friction="200"/>
+            <dynamics damping="50" friction="150"/>
             <axis xyz="0 0 1"/>
             <limit lower="${-90 * d2r}" upper="${60 * d2r}" velocity=".15" effort="300"/>
-            <!-- <limit lower="${-90 * d2r}" upper="${60 * d2r}" velocity=".13" effort="1000"/> -->
         </joint>
         <xacro:simple_transmission joint="${namespace}/elbow" />
@@ -181,7 +178,8 @@
             <origin xyz="0.1349014 -0.1936267 0" rpy="${0.5*PI} 0 0"/>
             <axis xyz="0 0 1"/>
-            <dynamics damping="50" friction="200"/>
-            <!-- <limit lower="${-135 * d2r}" upper="${135 * d2r}" velocity=".15" effort="200"/> -->
+            <dynamics damping="300" friction="1000"/>
+            <!-- <dynamics damping="300" friction="400"/> -->
             <limit lower="${-135 * d2r}" upper="${135 * d2r}" velocity=".25" effort="1000"/>
+            <!-- <limit lower="${-135 * d2r}" upper="${135 * d2r}" velocity=".25" effort="800"/> -->
         </joint>
         <xacro:simple_transmission joint="${namespace}/roll" />
@@ -212,7 +210,6 @@
             <origin xyz="0 0 0.31595760629823427" rpy="${-0.5*PI} ${-0.5*PI} 0"/>
             <axis xyz="0 0 1"/>
-            <dynamics damping="50" friction="200"/>
-            <limit lower="${-90 * d2r}" upper="${90 * d2r}" velocity=".26" effort="200"/>
-            <!-- <limit lower="${-90 * d2r}" upper="${90 * d2r}" velocity=".26" effort="1000"/> -->
+            <dynamics damping="10.0" friction="10.0"/>
+            <limit lower="${-90 * d2r}" upper="${90 * d2r}" velocity=".3" effort="50"/>
         </joint>
         <xacro:simple_transmission joint="${namespace}/pitch" />

Commit message: ADD New marker tags for BOP Panel FIX Oberon7 serial_arm parameters
Signed-off-by: Luiz Ricardo Douat <luizricardo.douat@de.bosch.com>

File: uuv_manipulators/oberon7/oberon7_description/urdf/serial_arm.xacro (robot description, xacro)
@@ -88,5 +88,6 @@
             <child link="${namespace}/shoulder_link"/>
             <axis xyz="0 0 1"/>
-            <dynamics damping="50" friction="200"/>
+            <!-- <dynamics damping="50" friction="200"/> -->
+            <dynamics damping="100" friction="150"/>
             <limit lower="${-60 * d2r}" upper="${60 * d2r}" velocity="0.17" effort="200"/>
             <!-- <limit lower="${-60 * d2r}" upper="${60 * d2r}" velocity="0.17" effort="1000"/> -->
@@ -119,5 +120,6 @@
             <origin xyz="0.06955 0.00015 0.01536" rpy="${0.5*pi} 0 0"/>
             <axis xyz="0 0 1"/>
-            <dynamics damping="50" friction="200"/>
+            <!-- <dynamics damping="50" friction="200"/> -->
+            <dynamics damping="50" friction="150"/>
             <limit lower="${-90 * d2r}" upper="${90 * d2r}" velocity=".17" effort="5000"/>
             <!-- <limit lower="${-90 * d2r}" upper="${90 * d2r}" velocity=".17" effort="1000"/> -->
@@ -149,5 +151,6 @@
             <child link="${namespace}/elbow_link"/>
             <origin xyz="0.55616 -0.01229 0" rpy="0 0 0"/>
-            <dynamics damping="50" friction="200"/>
+            <!-- <dynamics damping="50" friction="200"/> -->
+            <dynamics damping="50" friction="150"/>
             <axis xyz="0 0 1"/>
             <limit lower="${-90 * d2r}" upper="${60 * d2r}" velocity=".15" effort="300"/>
@@ -181,5 +184,6 @@
             <origin xyz="0.1349014 -0.1936267 0" rpy="${0.5*PI} 0 0"/>
             <axis xyz="0 0 1"/>
-            <dynamics damping="50" friction="200"/>
+            <!-- <dynamics damping="50" friction="200"/> -->
+            <dynamics damping="300" friction="1000"/>
             <!-- <limit lower="${-135 * d2r}" upper="${135 * d2r}" velocity=".15" effort="200"/> -->
             <limit lower="${-135 * d2r}" upper="${135 * d2r}" velocity=".25" effort="1000"/>
@@ -212,7 +216,8 @@
             <origin xyz="0 0 0.31595760629823427" rpy="${-0.5*PI} ${-0.5*PI} 0"/>
             <axis xyz="0 0 1"/>
-            <dynamics damping="50" friction="200"/>
-            <limit lower="${-90 * d2r}" upper="${90 * d2r}" velocity=".26" effort="200"/>
-            <!-- <limit lower="${-90 * d2r}" upper="${90 * d2r}" velocity=".26" effort="1000"/> -->
+            <!-- <dynamics damping="50" friction="200"/> -->
+            <dynamics damping="10" friction="10"/>
+            <!-- <limit lower="${-90 * d2r}" upper="${90 * d2r}" velocity=".26" effort="200"/> -->
+            <limit lower="${-90 * d2r}" upper="${90 * d2r}" velocity=".3" effort="50"/>
         </joint>
         <xacro:simple_transmission joint="${namespace}/pitch" />
