Commit message: rexrov_base: replace collision mesh with primitives
Signed-off-by: Sebastian Scherer <Sebastian.Scherer2@de.bosch.com>

File: uuv_descriptions/models/rexrov/urdf/rexrov_base.xacro (robot description, xacro)
@@ -26,5 +26,4 @@
   <xacro:property name="namespace" value="rexrov"/>
   <xacro:property name="visual_mesh_file" value="file://$(find uuv_descriptions)/models/rexrov/mesh/RexROV_no_props.dae"/>
-  <xacro:property name="collision_mesh_file" value="file://$(find uuv_descriptions)/models/rexrov/mesh/RexROV_no_props.stl"/>
   <xacro:property name="prop_mesh_file" value="file://$(find uuv_descriptions)/models/rexrov/mesh/prop.dae"/>
   <!-- Mass, see p.28 in Berg2012 -->
@@ -94,9 +93,24 @@
         </geometry>
       </visual>
-      <collision>
-        <origin xyz="0 0 0" rpy="0 0 0"/>
-        <geometry>
-          <mesh filename="${collision_mesh_file}" scale="1 1 1"/>
-        </geometry>
+      <!-- bottom plate -->
+      <collision>
+        <origin xyz="0 0 -0.75" rpy="0 0 0"/>
+        <geometry>
+          <box size="2.56 1.50 0.10"/>
+        </geometry>
+      </collision>
+      <!-- top plate -->
+      <collision>
+        <origin xyz="0 0 0.60" rpy="0 0 0"/>
+        <geometry><box size="2.56 1.50 0.40"/></geometry>
+      </collision>
+      <!-- left / right sides -->
+      <collision>
+        <origin xyz="-0.20 0.70 -0.15" rpy="0 0 0"/>
+        <geometry><box size="2.20 0.10 1.10"/></geometry>
+      </collision>
+      <collision>
+        <origin xyz="-0.20 -0.70 -0.15" rpy="0 0 0"/>
+        <geometry><box size="2.20 0.10 1.10"/></geometry>
       </collision>
     </link>

Commit message: MV RexROV underwater object plugin parameters to a new file.
Signed-off-by: Musa Morena Marcusso Manhães <Musa.Marcusso@de.bosch.com>

File: uuv_descriptions/models/rexrov/urdf/rexrov_base.xacro (robot description, xacro)
@@ -29,12 +29,7 @@
   <!-- Mass, see p.28 in Berg2012 -->
   <xacro:property name="mass" value="1862.87"/>
-  <!-- Volume, see p.31 in Berg2012 -->
-  <xacro:property name="volume" value="1.83826"/>
-  <!-- Center of buoyancy according to eq. (3.1) p. 28 in Berg2012.
-       The original values, [0.0822, -0.00773, 0.3872] however, seem to
-       assume NWU (otherwise cob is below cog?).  -->
-  <xacro:property name="cob" value="0.0 0.0 0.3"/>
   <!-- Thruster joint and link snippet -->
-  <xacro:macro name="thruster_macro" params="namespace thruster_id *origin">
+  <xacro:macro name="thruster_macro"
+               params="namespace thruster_id *origin">
     <joint name="${namespace}/thruster_${thruster_id}_joint" type="continuous">
       <xacro:insert_block name="origin"/>
@@ -78,5 +73,5 @@
     </gazebo>
   </xacro:macro>
-  <xacro:macro name="rexrov_base" params="namespace debug">
+  <xacro:macro name="rexrov_base" params="namespace debug *gazebo">
     <!-- base_link according to ROS conventions: x forward, z up -->
     <link name="${namespace}/base_link">
@@ -122,37 +117,7 @@
       <limit effort="0" lower="0" upper="0" velocity="0"/>
     </joint>
-    <!-- Set up hydrodynamic plugin -->
+    <!-- Set up hydrodynamic plugin given as input parameter -->
+    <xacro:insert_block name="gazebo"/>
     <gazebo>
-      <plugin name="uuv_plugin" filename="libunderwater_object_ros_plugin.so">
-        <fluid_density>1028.0</fluid_density>
-        <flow_velocity_topic>hydrodynamics/current_velocity</flow_velocity_topic>
-        <debug>${debug}</debug>
-        <link name="${namespace}/base_link">
-          <neutrally_buoyant>0</neutrally_buoyant>
-          <volume>${volume}</volume>
-          <box>
-            <width>1.5</width>
-            <length>2.6</length>
-            <height>1.6</height>
-          </box>
-          <center_of_buoyancy>${cob}</center_of_buoyancy>
-          <!-- Added mass: see p.28 in Berg2012 -->
-          <hydrodynamic_model>
-            <type>fossen</type>
-            <added_mass>
-               779.79 -6.8773 -103.32 8.5426 -165.54 -7.8033
-              -6.8773 1222 51.29 409.44 -5.8488 62.726
-                -103.32 51.29 3659.9 6.1112 -386.42 10.774
-                8.5426 409.44 6.1112 534.9 -10.027 21.019
-                -165.54 -5.8488 -386.42 -10.027 842.69 -1.1162
-                -7.8033 62.726 10.775 21.019 -1.1162 224.32
-            </added_mass>
-            <!-- Linear damping: see p.31 in Berg2012 -->
-            <linear_damping>-74.82 -69.48 -728.4 -268.8 -309.77 -105</linear_damping>
-            <!-- Non-linear damping: see p.30 in Berg2012 -->
-            <quadratic_damping>-748.22 -992.53 -1821.01 -672 -774.44 -523.27</quadratic_damping>
-          </hydrodynamic_model>
-        </link>
-      </plugin>
       <!-- optional: plugin to test compare Gazebo's returned accelerations
       <plugin name="${namespace}_test_plugin" filename="libaccelerations_test_plugin.so">

Commit message: Add April_tag and Noisy sensor
Signed-off-by: Luiz Ricardo Douat <luizricardo.douat@de.bosch.com>

File: uuv_descriptions/models/rexrov/urdf/rexrov_base.xacro (robot description, xacro)
@@ -150,5 +150,5 @@
       <origin xyz="0.412125 -0.505415 0.129" rpy="${0*d2r} ${0*d2r} ${-135*d2r}"/>
     </xacro:thruster_macro>
-    <!-- Mount a 3D pose sensor -->
+    <!-- Mount a 3D pose sensor (Groung truth values) -->
     <link name="${namespace}/pose_sensor_link">
       <xacro:box_inertial x="0" y="0" z="0" mass="0.01">
@@ -176,4 +176,33 @@
         <frameName>world</frameName>
         <gaussianNoise>0.0</gaussianNoise>
+        <updateRate>30</updateRate>
+      </plugin>
+    </gazebo>
+    <!-- Mount a noisy 3D pose sensor -->
+    <link name="${namespace}/pose_noisy_sensor_link">
+      <xacro:box_inertial x="0" y="0" z="0" mass="0.01">
+        <origin xyz="0 0 0" rpy="0 0 0"/>
+      </xacro:box_inertial>
+      <visual>
+        <geometry>
+          <box size="0.1 0.1 0.1"/>
+        </geometry>
+      </visual>
+      <xacro:no_collision/>
+    </link>
+    <joint name="${namespace}/pose_noisy_sensor_joint" type="revolute">
+      <origin xyz="0 0 0" rpy="0 0 0"/>
+      <axis xyz="0 0 1"/>
+      <parent link="${namespace}/base_link"/>
+      <child link="${namespace}/pose_noisy_sensor_link"/>
+      <limit effort="0" lower="0" upper="0" velocity="0"/>
+    </joint>
+    <gazebo>
+      <plugin name="pose_noise_3d_plugin" filename="libgazebo_ros_p3d.so">
+        <robotNamespace>${namespace}</robotNamespace>
+        <bodyName>${namespace}/base_link</bodyName>
+        <topicName>pose_noisy</topicName>
+        <frameName>world</frameName>
+        <gaussianNoise>0.02</gaussianNoise>
         <updateRate>30</updateRate>
       </plugin>

Commit message: RM Ned link, transformations now computed in the plugin
Signed-off-by: Musa Morena Marcusso Manhaes <Musa.Marcusso@de.bosch.com>

File: uuv_descriptions/models/rexrov/urdf/rexrov_base.xacro (robot description, xacro)
@@ -110,12 +110,4 @@
       </collision>
     </link>
-    <xacro:dummy_link name="${namespace}/ned_link" />
-    <joint name="ned_joint" type="fixed">
-      <!-- This is revolute and not static since gazebo would remove ned_link -->
-      <origin xyz="0 0 0" rpy="${pi} 0 0"/>
-      <parent link="${namespace}/base_link"/>
-      <child link="${namespace}/ned_link"/>
-      <limit effort="0" lower="0" upper="0" velocity="0"/>
-    </joint>
     <!-- Set up hydrodynamic plugin given as input parameter -->
     <xacro:insert_block name="gazebo"/>
