Commit message: RM Redundant definition of PI
Signed-off-by: Musa Morena Marcusso Manhaes <Musa.Marcusso@de.bosch.com>

File: uuv_descriptions/models/common/urdf/common.urdf.xacro (robot description, xacro)
@@ -13,5 +13,4 @@
 -->
 <robot xmlns:xacro="http://www.ros.org/wiki/xacro" >
-  <xacro:property name="pi" value="3.14159"/>
   <!-- Conversion factor: radian = d2r*degrees -->
   <xacro:property name="d2r" value="0.01745329"/>

Commit message: MV Joint state publisher snippets
Now in misc.xacro from uuv_gazebo_ros_plugins

Signed-off-by: Musa Morena Marcusso Manhaes <Musa.Marcusso@de.bosch.com>

File: uuv_descriptions/models/common/urdf/common.urdf.xacro (robot description, xacro)
@@ -142,22 +142,3 @@
     </xacro:box_inertial>
   </xacro:macro>
-  <!-- Default joint state publisher -->
-  <xacro:macro name="default_joint_state_publisher" params="namespace update_rate">
-    <gazebo>
-      <plugin name="joint_state_publisher" filename="libjoint_state_publisher.so">
-        <robotNamespace>${namespace}</robotNamespace>
-        <updateRate>${update_rate}</updateRate>
-      </plugin>
-    </gazebo>
-  </xacro:macro>
-  <!-- Joint state publisher with moving joints -->
-  <xacro:macro name="custom_joint_state_publisher" params="namespace update_rate joints">
-    <gazebo>
-      <plugin name="joint_state_publisher" filename="libjoint_state_publisher.so">
-        <robotNamespace>${namespace}</robotNamespace>
-        <updateRate>${update_rate}</updateRate>
-        <movingJoints>${joints}</movingJoints>
-      </plugin>
-    </gazebo>
-  </xacro:macro>
 </robot>
