Commit message: RM Debug flag from rexrov_base macro.
Signed-off-by: Musa Morena Marcusso Manhães <Musa.Marcusso@de.bosch.com>

File: uuv_descriptions/models/rexrov/robots/rexrov_default.xacro (robot description, xacro)
@@ -19,5 +19,5 @@
   <xacro:include filename="$(find uuv_descriptions)/models/rexrov/urdf/rexrov.gazebo.xacro"/>
   <!-- Create the rexrov -->
-  <xacro:rexrov_base namespace="$(arg namespace)" debug="$(arg debug)">
+  <xacro:rexrov_base namespace="$(arg namespace)">
     <!-- The underwater object plugin is given as an input block parameter to
      allow the addition of external models of manipulator units -->

File: uuv_descriptions/models/rexrov/robots/rexrov_oberon4.xacro (robot description, xacro)
@@ -20,5 +20,5 @@
   <xacro:include filename="$(find oberon4_description)/robots/oberon4_default.xacro" />
   <!-- Create the ROV -->
-  <xacro:rexrov_base namespace="$(arg namespace)" debug="$(arg debug)">
+  <xacro:rexrov_base namespace="$(arg namespace)">
     <!-- The underwater object plugin is given as an input block parameter to
      allow the addition of external models of manipulator units -->

File: uuv_descriptions/models/rexrov/robots/rexrov_oberon_arms.xacro (robot description, xacro)
@@ -21,5 +21,5 @@
   <xacro:include filename="$(find oberon_description)/robots/oberon_parallel.xacro" />
   <!-- Create the ROV -->
-  <xacro:rexrov_base namespace="$(arg namespace)" debug="$(arg debug)">
+  <xacro:rexrov_base namespace="$(arg namespace)">
     <!-- The underwater object plugin is given as an input block parameter to
      allow the addition of external models of manipulator units -->

File: uuv_descriptions/models/rexrov/robots/rexrov_oberon_dummy.xacro (robot description, xacro)
@@ -19,5 +19,5 @@
   <xacro:include filename="$(find oberon_description)/robots/oberon_dummy.xacro" />
   <!-- Create the ROV -->
-  <xacro:rexrov_base namespace="$(arg namespace)" debug="$(arg debug)">
+  <xacro:rexrov_base namespace="$(arg namespace)">
     <!-- The underwater object plugin is given as an input block parameter to
      allow the addition of external models of manipulator units -->

File: uuv_descriptions/models/rexrov/robots/rexrov_oberon_parallel.xacro (robot description, xacro)
@@ -20,5 +20,5 @@
   <xacro:include filename="$(find oberon_description)/robots/oberon_parallel.xacro" />
   <!-- Create the ROV -->
-  <xacro:rexrov_base namespace="$(arg namespace)" debug="$(arg debug)">
+  <xacro:rexrov_base namespace="$(arg namespace)">
     <!-- The underwater object plugin is given as an input block parameter to
      allow the addition of external models of manipulator units -->

File: uuv_descriptions/models/rexrov/robots/rexrov_sonar.xacro (robot description, xacro)
@@ -18,6 +18,6 @@
   <xacro:include filename="$(find uuv_descriptions)/models/rexrov/urdf/rexrov_base.xacro"/>
   <xacro:include filename="$(find uuv_descriptions)/models/rexrov/urdf/rexrov.gazebo.xacro"/>
-  <!-- Create the rexrov -->
-  <xacro:rexrov_base namespace="$(arg namespace)" debug="$(arg debug)">
+  <!-- Create the RexROV vehicle -->
+  <xacro:rexrov_base namespace="$(arg namespace)">
     <!-- The underwater object plugin is given as an input block parameter to
      allow the addition of external models of manipulator units -->

File: uuv_descriptions/models/rexrov/urdf/rexrov_base.xacro (robot description, xacro)
@@ -24,6 +24,5 @@
   <xacro:include filename="$(find uuv_descriptions)/models/common/urdf/common.urdf.xacro"/>
   <xacro:include filename="$(find uuv_sensor_plugins_ros)/urdf/sensor_snippets.xacro"/>
-  <!-- parameters -->
-  <xacro:property name="debug" value="0"/>
+  <!-- Parameters -->
   <xacro:property name="namespace" value="rexrov"/>
   <xacro:property name="visual_mesh_file" value="file://$(find uuv_descriptions)/models/rexrov/mesh/RexROV_no_props.dae"/>
@@ -75,5 +74,5 @@
     </gazebo>
   </xacro:macro>
-  <xacro:macro name="rexrov_base" params="namespace debug *gazebo">
+  <xacro:macro name="rexrov_base" params="namespace *gazebo">
     <!-- base_link according to ROS conventions: x forward, z up -->
     <link name="${namespace}/base_link">

Commit message: CHANGE Source of sensor snippets and option for world_frame input
Signed-off-by: Musa Morena Marcusso Manhaes <Musa.Marcusso@de.bosch.com>

File: uuv_descriptions/models/rexrov/robots/rexrov_default.xacro (robot description, xacro)
@@ -15,9 +15,12 @@
   <xacro:arg name="debug" default="0"/>
   <xacro:arg name="namespace" default="rexrov"/>
+  <xacro:arg name="inertial_reference_frame" default="world"/>
   <!-- Include the ROV macro file -->
   <xacro:include filename="$(find uuv_descriptions)/models/rexrov/urdf/rexrov_base.xacro"/>
   <xacro:include filename="$(find uuv_descriptions)/models/rexrov/urdf/rexrov.gazebo.xacro"/>
   <!-- Create the rexrov -->
-  <xacro:rexrov_base namespace="$(arg namespace)">
+  <xacro:rexrov_base
+    namespace="$(arg namespace)"
+    inertial_reference_frame="$(arg inertial_reference_frame)">
     <!-- The underwater object plugin is given as an input block parameter to
      allow the addition of external models of manipulator units -->

File: uuv_descriptions/models/rexrov/robots/rexrov_default_noisy_pose.xacro (robot description, xacro)
@@ -16,9 +16,12 @@
   <xacro:arg name="namespace" default="rexrov"/>
   <xacro:arg name="noise" default="0.02"/>
+  <xacro:arg name="inertial_reference_frame" default="world"/>
   <!-- Include the ROV macro file -->
   <xacro:include filename="$(find uuv_descriptions)/models/rexrov/urdf/rexrov_base.xacro"/>
   <xacro:include filename="$(find uuv_descriptions)/models/rexrov/urdf/rexrov.gazebo.xacro"/>
   <!-- Create the rexrov -->
-  <xacro:rexrov_base namespace="$(arg namespace)">
+  <xacro:rexrov_base
+    namespace="$(arg namespace)"
+    inertial_reference_frame="$(arg inertial_reference_frame)">
     <!-- The underwater object plugin is given as an input block parameter to
      allow the addition of external models of manipulator units -->

File: uuv_descriptions/models/rexrov/robots/rexrov_oberon4.xacro (robot description, xacro)
@@ -15,4 +15,5 @@
   <xacro:arg name="debug" default="0"/>
   <xacro:arg name="namespace" default="rexrov"/>
+  <xacro:arg name="inertial_reference_frame" default="world"/>
   <!-- Include the ROV macro file -->
   <xacro:include filename="$(find uuv_descriptions)/models/rexrov/urdf/rexrov_base.xacro"/>
@@ -20,5 +21,7 @@
   <xacro:include filename="$(find oberon4_description)/robots/oberon4_default.xacro" />
   <!-- Create the ROV -->
-  <xacro:rexrov_base namespace="$(arg namespace)">
+  <xacro:rexrov_base
+    namespace="$(arg namespace)"
+    inertial_reference_frame="$(arg inertial_reference_frame)">
     <!-- The underwater object plugin is given as an input block parameter to
      allow the addition of external models of manipulator units -->

File: uuv_descriptions/models/rexrov/robots/rexrov_oberon7.xacro (robot description, xacro)
@@ -15,4 +15,5 @@
   <xacro:arg name="debug" default="0"/>
   <xacro:arg name="namespace" default="rexrov"/>
+  <xacro:arg name="inertial_reference_frame" default="world"/>
   <!-- Include the ROV macro file -->
   <xacro:include filename="$(find uuv_descriptions)/models/rexrov/urdf/rexrov_base.xacro"/>
@@ -20,5 +21,7 @@
   <xacro:include filename="$(find oberon7_description)/robots/oberon7_default.xacro" />
   <!-- Create the ROV -->
-  <xacro:rexrov_base namespace="$(arg namespace)">
+  <xacro:rexrov_base
+    namespace="$(arg namespace)"
+    inertial_reference_frame="$(arg inertial_reference_frame)">
     <!-- The underwater object plugin is given as an input block parameter to
      allow the addition of external models of manipulator units -->

File: uuv_descriptions/models/rexrov/robots/rexrov_oberon_arms.xacro (robot description, xacro)
@@ -15,4 +15,5 @@
   <xacro:arg name="debug" default="0"/>
   <xacro:arg name="namespace" default="rexrov"/>
+  <xacro:arg name="inertial_reference_frame" default="world"/>
   <!-- Include the ROV macro file -->
   <xacro:include filename="$(find uuv_descriptions)/models/rexrov/urdf/rexrov_base.xacro"/>
@@ -21,5 +22,7 @@
   <xacro:include filename="$(find oberon7_description)/robots/oberon7_default.xacro" />
   <!-- Create the ROV -->
-  <xacro:rexrov_base namespace="$(arg namespace)">
+  <xacro:rexrov_base
+    namespace="$(arg namespace)"
+    inertial_reference_frame="$(arg inertial_reference_frame)">
     <!-- The underwater object plugin is given as an input block parameter to
      allow the addition of external models of manipulator units -->

File: uuv_descriptions/models/rexrov/robots/rexrov_sonar.xacro (robot description, xacro)
@@ -15,9 +15,12 @@
   <xacro:arg name="debug" default="0"/>
   <xacro:arg name="namespace" default="rexrov"/>
+  <xacro:arg name="inertial_reference_frame" default="world"/>
   <!-- Include the ROV macro file -->
   <xacro:include filename="$(find uuv_descriptions)/models/rexrov/urdf/rexrov_base.xacro"/>
   <xacro:include filename="$(find uuv_descriptions)/models/rexrov/urdf/rexrov.gazebo.xacro"/>
   <!-- Create the RexROV vehicle -->
-  <xacro:rexrov_base namespace="$(arg namespace)">
+  <xacro:rexrov_base
+    namespace="$(arg namespace)"
+    inertial_reference_frame="$(arg inertial_reference_frame)">
     <!-- The underwater object plugin is given as an input block parameter to
      allow the addition of external models of manipulator units -->

File: uuv_descriptions/models/rexrov/urdf/rexrov_base.xacro (robot description, xacro)
@@ -23,6 +23,7 @@
   <!-- includes -->
   <xacro:include filename="$(find uuv_descriptions)/models/common/urdf/common.urdf.xacro"/>
-  <xacro:include filename="$(find uuv_sensor_plugins_ros)/urdf/sensor_snippets.xacro"/>
+  <xacro:include filename="$(find uuv_sensor_ros_plugins)/urdf/sensor_snippets.xacro"/>
   <xacro:include filename="$(find uuv_gazebo_ros_plugins)/urdf/snippets.xacro"/>
+  <xacro:include filename="$(find uuv_sensor_plugins_ros)/urdf/imu_snippets.xacro"/>
   <!-- Parameters -->
   <xacro:property name="namespace" value="rexrov"/>
@@ -31,5 +32,5 @@
   <!-- Mass, see p.28 in Berg2012 -->
   <xacro:property name="mass" value="1862.87"/>
-  <xacro:macro name="rexrov_base" params="namespace *gazebo">
+  <xacro:macro name="rexrov_base" params="namespace *gazebo inertial_reference_frame">
     <!-- base_link according to ROS conventions: x forward, z up -->
     <link name="${namespace}/base_link">

File: uuv_descriptions/models/rexrov/urdf/rexrov_sensors.xacro (robot description, xacro)
@@ -14,7 +14,12 @@
 <robot xmlns:xacro="http://www.ros.org/wiki/xacro">
   <!-- DVL  -->
-  <xacro:default_dvl namespace="${namespace}" parent_link="${namespace}/base_link">
+  <xacro:default_dvl_macro
+    namespace="${namespace}"
+    parent_link="${namespace}/base_link"
+    inertial_reference_frame="${inertial_reference_frame}">
     <origin xyz="-1.4 0 -0.312" rpy="0 ${0.5*pi} 0"/>
-  </xacro:default_dvl>
+  </xacro:default_dvl_macro>
+  <!-- Magnetometer  -->
+  <xacro:default_magnetometer namespace="${namespace}" parent_link="${namespace}/base_link"/>
   <!-- RPT  -->
   <xacro:default_rpt namespace="${namespace}" parent_link="${namespace}/base_link">
@@ -22,11 +27,14 @@
   </xacro:default_rpt>
   <!-- Pressure  -->
-  <xacro:default_pressure namespace="${namespace}" parent_link="${namespace}/base_link">
+  <xacro:default_pressure_macro namespace="${namespace}" parent_link="${namespace}/base_link">
     <origin xyz="-1.32 0.5 0.85" rpy="0 0 0"/>
-  </xacro:default_pressure>
+  </xacro:default_pressure_macro>
   <!-- IMU  -->
-  <xacro:default_imu namespace="${namespace}" parent_link="${namespace}/base_link">
+  <xacro:default_imu_macro
+    namespace="${namespace}"
+    parent_link="${namespace}/base_link"
+    inertial_reference_frame="${inertial_reference_frame}">
     <origin xyz="0 0 0" rpy="0 0 0"/>
-  </xacro:default_imu>
+  </xacro:default_imu_macro>
   <!-- Mount a camera -->
   <xacro:default_camera namespace="${namespace}" parent_link="${namespace}/base_link" suffix="">
@@ -42,4 +50,7 @@
   <xacro:default_gps namespace="${namespace}" parent_link="${namespace}/base_link" />
   <!-- Mount a Pose 3D sensor. -->
-  <xacro:default_pose_3d namespace="${namespace}" parent_link="${namespace}/base_link" />
+  <xacro:default_pose_3d_macro
+    namespace="${namespace}"
+    parent_link="${namespace}/base_link"
+    inertial_reference_frame="${inertial_reference_frame}" />
 </robot>
