Commit message: ADD Joint state publisher snippet to misc.xacro
Signed-off-by: Musa Morena Marcusso Manhaes <Musa.Marcusso@de.bosch.com>

File: uuv_gazebo_plugins/uuv_gazebo_ros_plugins/urdf/misc.xacro (robot description, xacro)
@@ -8,3 +8,12 @@
     </gazebo>
   </xacro:macro>
+  <!-- Default joint state publisher -->
+  <xacro:macro name="default_joint_state_publisher" params="namespace update_rate">
+    <gazebo>
+      <plugin name="joint_state_publisher" filename="libjoint_state_publisher.so">
+        <robotNamespace>${namespace}</robotNamespace>
+        <updateRate>${update_rate}</updateRate>
+      </plugin>
+    </gazebo>
+  </xacro:macro>
 </robot>
