Commit message: FIX Typo in fin macro snippet
Signed-off-by: Musa Morena Marcusso Manhaes <Musa.Marcusso@de.bosch.com>

File: uuv_gazebo_plugins/uuv_gazebo_ros_plugins/urdf/fin_snippets.xacro (robot description, xacro)
@@ -74,5 +74,5 @@
             current_velocity_topic">
     <joint name="${namespace}/fin${fin_id}_joint" type="revolute">
-        <limit effort="0" lower="${min_joint_limi}" upper="${max_joint_limit}" velocity="0"/>
+        <limit effort="0" lower="${min_joint_limit}" upper="${max_joint_limit}" velocity="0"/>
         <xacro:insert_block name="origin"/>
         <axis xyz="0 0 1"/>
