Commit message: ADD More snippet options for ENU and NED frame
Signed-off-by: Musa Morena Marcusso Manhaes <Musa.Marcusso@de.bosch.com>

File: uuv_sensor_plugins/uuv_sensor_ros_plugins/urdf/dvl_snippets.xacro (robot description, xacro)
@@ -21,4 +21,33 @@
     </collision>
   </xacro:macro>
+  <xacro:macro name="default_dvl_macro" params="namespace parent_link *origin inertial_reference_frame">
+    <xacro:dvl_plugin_macro
+      namespace="${namespace}"
+      suffix=""
+      parent_link="${parent_link}"
+      reference_frame="${inertial_reference_frame}"
+      update_rate="7"
+      topic="dvl"
+      scale="1">
+      <xacro:insert_block name="origin" />
+    </xacro:dvl_plugin_macro>
+  </xacro:macro>
+  <xacro:macro name="default_dvl_sensor_enu" params="namespace parent_link *origin">
+    <xacro:default_dvl_macro
+      namespace="${namespace}"
+      parent_link="${parent_link}"
+      reference_frame="world">
+      <xacro:insert_block name="origin" />
+    </xacro:default_dvl_macro>
+  </xacro:macro>
+  <xacro:macro name="default_dvl_sensor_ned" params="namespace parent_link *origin">
+    <xacro:default_dvl_macro
+      namespace="${namespace}"
+      parent_link="${parent_link}"
+      reference_frame="world_ned">
+      <xacro:insert_block name="origin" />
+    </xacro:default_dvl_macro>
+  </xacro:macro>
+  <!-- DEPRECATED MACRO: See default_dvl_sensor_enu -->
   <xacro:macro name="default_dvl" params="namespace parent_link *origin">
     <xacro:dvl_plugin_macro
@@ -26,4 +55,5 @@
       suffix=""
       parent_link="${parent_link}"
+      reference_frame="world"
       update_rate="7"
       topic="dvl"
@@ -87,5 +117,5 @@
   </xacro:macro>
   <xacro:macro name="dvl_plugin_macro" params="namespace suffix parent_link topic
-    scale *origin update_rate">
+    scale *origin update_rate reference_frame">
     <link name="${namespace}/dvl${suffix}_link">
       <inertial>
@@ -133,4 +163,5 @@
         <enable_gazebo_messages>false</enable_gazebo_messages>
         <enable_local_ned_frame>false</enable_local_ned_frame>
+        <static_reference_frame>${reference_frame}</static_reference_frame>
         <!-- Declaring the beams -->
         <beam_link_name_0>${namespace}/dvl_sonar0_link</beam_link_name_0>

File: uuv_sensor_plugins/uuv_sensor_ros_plugins/urdf/pose_3d_snippets.xacro (robot description, xacro)
@@ -44,5 +44,4 @@
   <xacro:macro name="pose_3d_sensor" params="namespace suffix parent_link
     gaussian_noise_sigma topic">
-    <!-- Default GPS. -->
     <xacro:pose_3d_macro
       namespace="${namespace}"
@@ -57,5 +56,4 @@
   </xacro:macro>
   <xacro:macro name="default_pose_3d" params="namespace parent_link">
-    <!-- Default GPS. -->
     <xacro:pose_3d_macro
       namespace="${namespace}"
@@ -69,20 +67,17 @@
     </xacro:pose_3d_macro>
   </xacro:macro>
-  <xacro:macro name="pose_3d_sensor_ned" params="namespace suffix parent_link
-    gaussian_noise_sigma topic">
-    <!-- Default GPS. -->
+  <xacro:macro name="default_pose_3d_enu" params="namespace parent_link">
     <xacro:pose_3d_macro
       namespace="${namespace}"
       parent_link="${parent_link}"
-      topic="${topic}"
+      topic="pose_gt"
       update_rate="20"
-      noise_sigma="${gaussian_noise_sigma}"
-      suffix="${suffix}"
-      reference_frame="world_ned">
+      noise_sigma="0.0"
+      suffix="default"
+      reference_frame="world">
       <origin xyz="0 0 0" rpy="0 0 0" />
     </xacro:pose_3d_macro>
   </xacro:macro>
   <xacro:macro name="default_pose_3d_ned" params="namespace parent_link">
-    <!-- Default GPS. -->
     <xacro:pose_3d_macro
       namespace="${namespace}"
@@ -96,3 +91,17 @@
     </xacro:pose_3d_macro>
   </xacro:macro>
+  <xacro:macro name="default_pose_3d_macro" params="namespace parent_link inertial_reference_frame">
+    <xacro:if value="${inertial_reference_frame == 'world'}">
+      <xacro:default_pose_3d_enu
+        namespace="${namespace}"
+        parent_link="${parent_link}">
+      </xacro:default_pose_3d_enu>
+    </xacro:if>
+    <xacro:if value="${inertial_reference_frame == 'world_ned'}">
+      <xacro:default_pose_3d_ned
+        namespace="${namespace}"
+        parent_link="${parent_link}">
+      </xacro:default_pose_3d_ned>
+    </xacro:if>
+  </xacro:macro>
 </robot>

File: uuv_sensor_plugins/uuv_sensor_ros_plugins/urdf/pressure_snippets.xacro (robot description, xacro)
@@ -20,4 +20,21 @@
       <origin xyz="0 0 0" rpy="0 ${0.5*pi} 0"/>
     </collision>
+  </xacro:macro>
+  <xacro:macro name="default_pressure_macro" params="namespace parent_link *origin">
+    <xacro:pressure_plugin_macro
+      namespace="${namespace}"
+      suffix=""
+      parent_link="${parent_link}"
+      topic="pressure"
+      mass="0.015"
+      update_rate="10"
+      range="30000"
+      stddev="3.0"
+      estimateDepth="false"
+      standardPressure="101.325"
+      kPaPerM="9.80638">
+      <inertia ixx="0.00001" ixy="0.0" ixz="0.0" iyy="0.00001" iyz="0.0" izz="0.00001" />
+      <xacro:insert_block name="origin" />>
+    </xacro:pressure_plugin_macro>
   </xacro:macro>
   <xacro:macro name="default_pressure" params="namespace parent_link *origin">

Commit message: Changed dvl_snippets.xacro so that all dvl topics publish at nominated update_rate. Signed-off-by: Fletcher F Thompson <fletcherthompsonx@gmail.com>

File: uuv_sensor_plugins/uuv_sensor_ros_plugins/urdf/dvl_snippets.xacro (robot description, xacro)
@@ -66,5 +66,5 @@
     </xacro:dvl_plugin_macro>
   </xacro:macro>
-  <xacro:macro name="dvl_single_sonar" params="namespace suffix index pitch yaw">
+  <xacro:macro name="dvl_single_sonar" params="namespace suffix index pitch yaw update_rate">
     <link name="${namespace}/dvl${suffix}_sonar${index}_link">
       <inertial>
@@ -85,5 +85,5 @@
       <sensor type="ray" name="dvl${suffix}_sonar${index}">
         <pose>0 0 0 0 0 0</pose>
-        <update_rate>1</update_rate>
+        <update_rate>${update_rate}</update_rate>
         <visualize>false</visualize>
         <ray>
@@ -111,5 +111,5 @@
           <gaussianNoise>0.005</gaussianNoise>
           <alwaysOn>true</alwaysOn>
-          <updateRate>1</updateRate>
+          <updateRate>${update_rate}</updateRate>
           <topicName>${topic}_sonar${index}</topicName>
           <frameName>${namespace}/dvl${suffix}_sonar${index}_link</frameName>
@@ -145,17 +145,17 @@
     <xacro:dvl_single_sonar
       namespace="${namespace}" suffix=""
-      index="0" pitch="-0.52" yaw="0.0">
+      index="0" pitch="-0.52" yaw="0.0" update_rate="${update_rate}">
     </xacro:dvl_single_sonar>
     <xacro:dvl_single_sonar
       namespace="${namespace}" suffix=""
-      index="1" pitch="0" yaw="0.52">
+      index="1" pitch="0" yaw="0.52" update_rate="${update_rate}">
     </xacro:dvl_single_sonar>
     <xacro:dvl_single_sonar
       namespace="${namespace}" suffix=""
-      index="2" pitch="0.52" yaw="0.0">
+      index="2" pitch="0.52" yaw="0.0" update_rate="${update_rate}">
     </xacro:dvl_single_sonar>
     <xacro:dvl_single_sonar
       namespace="${namespace}" suffix=""
-      index="3" pitch="0.0" yaw="-0.52">
+      index="3" pitch="0.0" yaw="-0.52" update_rate="${update_rate}">
     </xacro:dvl_single_sonar>
     <gazebo>
