Commit message: FIX Path to sensor meshes
Signed-off-by: Musa Morena Marcusso Manhaes <Musa.Marcusso@de.bosch.com>

File: uuv_sensor_plugins/uuv_sensor_ros_plugins/urdf/camera_snippets.xacro (robot description, xacro)
@@ -69,5 +69,5 @@
       <visual>
         <geometry>
-          <mesh filename="file://$(find uuv_sensor_plugins)/mesh/oe14-372.dae" scale="${scale} ${scale} ${scale}"/>
+          <mesh filename="file://$(find uuv_sensor_ros_plugins)/meshes/oe14-372.dae" scale="${scale} ${scale} ${scale}"/>
         </geometry>
       </visual>
@@ -154,5 +154,5 @@
       <visual>
         <geometry>
-          <mesh filename="file://$(find uuv_sensor_plugins)/mesh/oe14-372.dae" scale="1 1 1"/>
+          <mesh filename="file://$(find uuv_sensor_ros_plugins)/meshes/oe14-372.dae" scale="1 1 1"/>
         </geometry>
       </visual>

File: uuv_sensor_plugins/uuv_sensor_ros_plugins/urdf/dvl_snippets.xacro (robot description, xacro)
@@ -126,5 +126,5 @@
       <visual>
         <geometry>
-          <mesh filename="file://$(find uuv_sensor_plugins)/mesh/dvl.dae" scale="${scale} ${scale} ${scale}"/>
+          <mesh filename="file://$(find uuv_sensor_ros_plugins)/meshes/dvl.dae" scale="${scale} ${scale} ${scale}"/>
         </geometry>
       </visual>

File: uuv_sensor_plugins/uuv_sensor_ros_plugins/urdf/rpt_snippets.xacro (robot description, xacro)
@@ -39,5 +39,5 @@
       <visual>
         <geometry>
-          <mesh filename="file://$(find uuv_sensor_plugins)/mesh/rpt.dae" scale="1 1 1"/>
+          <mesh filename="file://$(find uuv_sensor_ros_plugins)/meshes/rpt.dae" scale="1 1 1"/>
         </geometry>
       </visual>

File: uuv_sensor_plugins/uuv_sensor_ros_plugins/urdf/sonar_snippets.xacro (robot description, xacro)
@@ -66,5 +66,5 @@
       <visual>
         <geometry>
-          <mesh filename="file://$(find uuv_sensor_plugins)/mesh/m450-130.dae" scale="1 1 1"/>
+          <mesh filename="file://$(find uuv_sensor_ros_plugins)/meshes/m450-130.dae" scale="1 1 1"/>
         </geometry>
       </visual>
@@ -89,5 +89,5 @@
       <visual>
         <geometry>
-          <mesh filename="file://$(find uuv_sensor_plugins)/mesh/p900.dae" scale="1 1 1"/>
+          <mesh filename="file://$(find uuv_sensor_ros_plugins)/meshes/p900.dae" scale="1 1 1"/>
         </geometry>
       </visual>

File: uuv_sensor_plugins/uuv_sensor_ros_plugins/urdf/stereo_snippets.xacro (robot description, xacro)
@@ -41,5 +41,5 @@
       <visual>
         <geometry>
-          <mesh filename="file://$(find uuv_sensor_plugins)/mesh/duo3d.dae"/>
+          <mesh filename="file://$(find uuv_sensor_ros_plugins)/meshes/duo3d.dae"/>
         </geometry>
       </visual>

Commit message: Fix to include an optical frame for the underwater camera plugin. Signed-off-by: Fletcher F Thompson <fletcherthompsonx@gmail.com>

File: uuv_sensor_plugins/uuv_sensor_ros_plugins/urdf/camera_snippets.xacro (robot description, xacro)
@@ -166,4 +166,24 @@
       <limit upper="0" lower="0" effort="0" velocity="0" />
     </joint>
+    <link name="${namespace}/camera${suffix}_link_optical">
+      <xacro:box_inertial x="0.0001" y="0.0001" z="0.0001" mass="0.001">
+        <origin xyz="0 0 0" rpy="0 0 0"/>
+      </xacro:box_inertial>
+      <collision>
+        <!-- todo: gazebo needs a collision volume or it will ignore the pose of
+           the joint that leads to this link (and assume it to be the identity) -->
+        <geometry>
+          <cylinder length="0.000001" radius="0.000001"/>
+        </geometry>
+        <origin xyz="0 0 0" rpy="0 ${0.5*pi} 0"/>
+      </collision>
+    </link>
+    <joint name="${namespace}/camera${suffix}_optical_joint" type="revolute">
+      <origin xyz="0 0 0" rpy="${-pi/2} 0 ${-pi/2}"/>
+      <parent link="${namespace}/camera${suffix}_link"/>
+      <child link="${namespace}/camera${suffix}_link_optical"/>
+      <limit upper="0" lower="0" effort="0" velocity="0" />
+      <axis xyz="1 0 0"/>
+    </joint>
     <gazebo reference="${namespace}/camera${suffix}_link">
       <sensor type="depth" name="camera${suffix}">
