Commit message: ADD Different noise models for the base plugins

File: uuv_sensor_plugins/uuv_sensor_ros_plugins/urdf/chemical_concentration_snippets.xacro (robot description, xacro)
@@ -30,4 +30,5 @@
       gamma="0.001"
       noise_sigma="0"
+      noise_amplitude="0"
       radius="3.0">
       <xacro:insert_block name="origin" />
@@ -70,4 +71,5 @@
       gain="1.0"
       noise_sigma="0"
+      noise_amplitude="0"
       radius="3.0">
       <xacro:insert_block name="origin" />
@@ -77,5 +79,5 @@
     params="namespace parent_link *origin suffix input_topic output_topic
             gamma radius update_rate reference_frame water_salinity_value plume_salinity_value
-            salinity_output_topic salinity_unit gain noise_sigma">
+            salinity_output_topic salinity_unit gain noise_sigma noise_amplitude">
     <!-- Sensor link -->
    <link name="${namespace}/cc_sensor_link">
@@ -112,4 +114,5 @@
        <gain>${gain}</gain>
        <noise_sigma>${noise_sigma}</noise_sigma>
+       <noise_amplitude>${noise_amplitude}</noise_amplitude>
      </plugin>
    </gazebo>

File: uuv_sensor_plugins/uuv_sensor_ros_plugins/urdf/dvl_snippets.xacro (robot description, xacro)
@@ -29,4 +29,6 @@
       update_rate="7"
       topic="dvl"
+      noise_sigma="0"
+      noise_amplitude="0"
       scale="1">
       <xacro:insert_block name="origin" />
@@ -58,4 +60,6 @@
       update_rate="7"
       topic="dvl"
+      noise_sigma="0"
+      noise_amplitude="0"
       scale="1">
       <xacro:insert_block name="origin" />
@@ -116,6 +120,7 @@
     </gazebo>
   </xacro:macro>
-  <xacro:macro name="dvl_plugin_macro" params="namespace suffix parent_link topic
-    scale *origin update_rate reference_frame">
+  <xacro:macro name="dvl_plugin_macro"
+    params="namespace suffix parent_link topic scale *origin update_rate
+    reference_frame noise_sigma noise_amplitude">
     <link name="${namespace}/dvl${suffix}_link">
       <inertial>
@@ -160,5 +165,6 @@
         <sensor_topic>${topic}</sensor_topic> <!-- (string): name of the sensor output topic and prefix of service names -->
         <update_rate>${update_rate}</update_rate> <!-- Update period [s] -->
-        <gaussian_noise_sigma>0.001</gaussian_noise_sigma> <!-- std dev of position estimates in x, y, z [m/s] -->
+        <noise_sigma>${noise_sigma}</noise_sigma> <!-- std dev of position estimates in x, y, z [m/s] -->
+        <noise_amplitude>${noise_amplitude}</noise_amplitude>
         <enable_gazebo_messages>false</enable_gazebo_messages>
         <enable_local_ned_frame>false</enable_local_ned_frame>

File: uuv_sensor_plugins/uuv_sensor_ros_plugins/urdf/magnetometer_snippets.xacro (robot description, xacro)
@@ -34,4 +34,5 @@
       noise_xy="1.0"
       noise_z="1.4"
+      noise_amplitude="0"
       turn_on_bias="2.0">
       <inertia ixx="0.00001" ixy="0.0" ixz="0.0" iyy="0.00001" iyz="0.0" izz="0.00001" />
@@ -42,5 +43,5 @@
   <xacro:macro name="magnetometer_plugin_macro"
     params="namespace suffix parent_link topic mass update_rate
-      mag_intensity noise_xy noise_z turn_on_bias
+      mag_intensity noise_xy noise_z turn_on_bias noise_amplitude
       *inertia *origin">
     <!-- Sensor link -->
@@ -79,4 +80,5 @@
         <noise_z>${noise_z}</noise_z> <!-- Discrete-time std. dev. of output noise in z-axis [muT] -->
         <turn_on_bias>${turn_on_bias}</turn_on_bias> <!-- Std. dev. of turn-on-bias [muT] -->
+        <noise_amplitude>${noise_amplitude}</noise_amplitude>
         <enable_gazebo_messages>false</enable_gazebo_messages>
         <enable_local_ned_frame>false</enable_local_ned_frame>

File: uuv_sensor_plugins/uuv_sensor_ros_plugins/urdf/pose_3d_snippets.xacro (robot description, xacro)
@@ -14,5 +14,5 @@
 <robot xmlns:xacro="http://www.ros.org/wiki/xacro">
   <xacro:macro name="pose_3d_macro" params="namespace suffix parent_link topic
-    update_rate *origin noise_sigma reference_frame publish_ned_odom">
+    update_rate *origin noise_sigma reference_frame publish_ned_odom noise_amplitude">
     <!-- Mount a 3D pose sensor -->
     <link name="${namespace}/pose_sensor_link_${suffix}">
@@ -36,5 +36,6 @@
         <sensor_topic>${topic}</sensor_topic>
         <static_reference_frame>${reference_frame}</static_reference_frame>
-        <gaussian_noise_sigma>${noise_sigma}</gaussian_noise_sigma>
+        <noise_sigma>${noise_sigma}</noise_sigma>
+        <noise_amplitude>${noise_amplitude}</noise_amplitude>
         <update_rate>${update_rate}</update_rate>
         <enable_gazebo_messages>false</enable_gazebo_messages>
@@ -44,5 +45,5 @@
   </xacro:macro>
   <xacro:macro name="pose_3d_sensor" params="namespace suffix parent_link
-    gaussian_noise_sigma topic">
+    gaussian_noise_sigma gaussian_noise_amplitude topic">
     <xacro:pose_3d_macro
       namespace="${namespace}"
@@ -51,4 +52,5 @@
       update_rate="20"
       noise_sigma="${gaussian_noise_sigma}"
+      noise_amplitude="${gaussian_noise_amplitude}"
       suffix="${suffix}"
       reference_frame="world"
@@ -64,4 +66,5 @@
       update_rate="20"
       noise_sigma="0.0"
+      noise_amplitude="0.0"
       suffix="default"
       reference_frame="world"
@@ -77,4 +80,5 @@
       update_rate="20"
       noise_sigma="0.0"
+      noise_amplitude="0.0"
       suffix="default"
       reference_frame="world"
@@ -90,4 +94,5 @@
       update_rate="20"
       noise_sigma="0.0"
+      noise_amplitude="0.0"
       suffix="default"
       reference_frame="world_ned"

File: uuv_sensor_plugins/uuv_sensor_ros_plugins/urdf/pressure_snippets.xacro (robot description, xacro)
@@ -30,5 +30,6 @@
       update_rate="10"
       range="30000"
-      stddev="3.0"
+      noise_sigma="3.0"
+      noise_amplitude="0.0"
       estimateDepth="false"
       standardPressure="101.325"
@@ -47,5 +48,6 @@
       update_rate="10"
       range="30000"
-      stddev="3.0"
+      noise_sigma="3.0"
+      noise_amplitude="0.0"
       estimateDepth="false"
       standardPressure="101.325"
@@ -57,5 +59,5 @@
   <xacro:macro name="pressure_plugin_macro"
     params="namespace suffix parent_link topic mass update_rate
-      range stddev estimateDepth standardPressure kPaPerM
+      range noise_sigma noise_amplitude estimateDepth standardPressure kPaPerM
       *inertia *origin">
     <link name="${namespace}/pressure${suffix}_link">
@@ -86,5 +88,6 @@
         <update_rate>${update_rate}</update_rate> <!-- Update period of accelerometer and gyroscope [s] -->
         <saturation>${range}</saturation> <!-- measurement range [kPa] -->
-        <noise_stddev>${stddev}</noise_stddev> <!-- measurement stddev [kPa] -->
+        <noise_sigma>${noise_sigma}</noise_sigma> <!-- measurement stddev [kPa] -->
+        <noise_amplitude>${noise_amplitude}</noise_amplitude>
         <estimate_depth_on>${estimateDepth}</estimate_depth_on> <!-- infer depth? -->
         <standard_pressure>${standardPressure}</standard_pressure> <!-- pressure at sea level (depth 0 m) [kPa] -->

File: uuv_sensor_plugins/uuv_sensor_ros_plugins/urdf/rpt_snippets.xacro (robot description, xacro)
@@ -26,9 +26,13 @@
       suffix=""
       parent_link="${parent_link}"
+      noise_amplitude="0.0"
+      noise_sigma="0.0"
       topic="rpt">
       <xacro:insert_block name="origin" />
     </xacro:rpt_plugin_macro>
   </xacro:macro>
-  <xacro:macro name="rpt_plugin_macro" params="namespace suffix parent_link topic *origin">
+  <xacro:macro name="rpt_plugin_macro"
+    params="namespace suffix parent_link topic noise_sigma noise_amplitude
+    *origin">
     <link name="${namespace}/rpt${suffix}_link">
       <inertial>
@@ -58,5 +62,6 @@
         <sensor_topic>${topic}</sensor_topic> <!-- name of the sensor output topic and prefix of service name -->
         <update_rate>0.5</update_rate> <!-- Update period [s] -->
-        <noise_std_dev>1.0</noise_std_dev> <!-- std dev of position estimates in x, y, z [m] -->
+        <noise_sigma>${noise_sigma}</noise_sigma> <!-- std dev of position estimates in x, y, z [m] -->
+        <noise_amplitude>${noise_amplitude}</noise_amplitude>
         <enable_gazebo_messages>false</enable_gazebo_messages>
       </plugin>

Commit message: stop warning mesg messages

File: uuv_sensor_plugins/uuv_sensor_ros_plugins/urdf/chemical_concentration_snippets.xacro (robot description, xacro)
@@ -44,10 +44,10 @@
     </xacro:default_chemical_concentration_sensor_macro>
   </xacro:macro>
-  <xacro:macro name="default_chemical_concentration_sensor_ned"
+  <xacro:macro name="default_chemical_concentration_sensor_aaa"
     params="namespace parent_link *origin">
     <xacro:default_chemical_concentration_sensor_macro
       namespace="${namespace}"
       parent_link="${parent_link}"
-      inertial_reference_frame="world_ned">
+      inertial_reference_frame="world_aaa">
       <xacro:insert_block name="origin" />
     </xacro:default_chemical_concentration_sensor_macro>
@@ -106,5 +106,5 @@
        <radius>${radius}</radius>
        <enable_gazebo_messages>false</enable_gazebo_messages>
-       <enable_local_ned_frame>false</enable_local_ned_frame>
+       <enable_local_aaa_frame>false</enable_local_aaa_frame>
        <static_reference_frame>${reference_frame}</static_reference_frame>
        <water_salinity_value>${water_salinity_value}</water_salinity_value>

File: uuv_sensor_plugins/uuv_sensor_ros_plugins/urdf/dvl_snippets.xacro (robot description, xacro)
@@ -43,9 +43,9 @@
     </xacro:default_dvl_macro>
   </xacro:macro>
-  <xacro:macro name="default_dvl_sensor_ned" params="namespace parent_link *origin">
+  <xacro:macro name="default_dvl_sensor_aaa" params="namespace parent_link *origin">
     <xacro:default_dvl_macro
       namespace="${namespace}"
       parent_link="${parent_link}"
-      reference_frame="world_ned">
+      reference_frame="world_aaa">
       <xacro:insert_block name="origin" />
     </xacro:default_dvl_macro>
@@ -168,5 +168,5 @@
         <noise_amplitude>${noise_amplitude}</noise_amplitude>
         <enable_gazebo_messages>false</enable_gazebo_messages>
-        <enable_local_ned_frame>false</enable_local_ned_frame>
+        <enable_local_aaa_frame>false</enable_local_aaa_frame>
         <static_reference_frame>${reference_frame}</static_reference_frame>
         <!-- Declaring the beams -->

File: uuv_sensor_plugins/uuv_sensor_ros_plugins/urdf/imu_snippets.xacro (robot description, xacro)
@@ -39,5 +39,5 @@
       accelerometer_turn_on_bias_sigma="0.1960"
       orientation_noise="0.01"
-      enable_local_ned_frame="false"
+      enable_local_aaa_frame="false"
       reference_frame="world"
       update_rate="50">
@@ -55,10 +55,10 @@
       </xacro:default_imu_enu>
     </xacro:if>
-    <xacro:if value="${inertial_reference_frame == 'world_ned'}">
-      <xacro:default_imu_ned
+    <xacro:if value="${inertial_reference_frame == 'world_aaa'}">
+      <xacro:default_imu_aaa
         namespace="${namespace}"
         parent_link="${parent_link}">
         <xacro:insert_block name="origin" />
-      </xacro:default_imu_ned>
+      </xacro:default_imu_aaa>
     </xacro:if>
   </xacro:macro>
@@ -80,5 +80,5 @@
       accelerometer_turn_on_bias_sigma="0.1960"
       orientation_noise="0.01"
-      enable_local_ned_frame="false"
+      enable_local_aaa_frame="false"
       reference_frame="world"
       update_rate="50">
@@ -87,5 +87,5 @@
     </xacro:imu_plugin_macro>
   </xacro:macro>
-  <xacro:macro name="default_imu_ned" params="namespace parent_link *origin">
+  <xacro:macro name="default_imu_aaa" params="namespace parent_link *origin">
     <!-- ADIS16448 IMU. -->
     <xacro:imu_plugin_macro
@@ -104,6 +104,6 @@
       accelerometer_turn_on_bias_sigma="0.1960"
       orientation_noise="0.01"
-      enable_local_ned_frame="true"
-      reference_frame="world_ned"
+      enable_local_aaa_frame="true"
+      reference_frame="world_aaa"
       update_rate="50">
       <inertia ixx="0.00001" ixy="0.0" ixz="0.0" iyy="0.00001" iyz="0.0" izz="0.00001" />
@@ -120,5 +120,5 @@
       orientation_noise
       update_rate reference_frame
-      enable_local_ned_frame
+      enable_local_aaa_frame
       *inertia *origin">
     <!-- IMU link -->
@@ -156,5 +156,5 @@
         <update_rate>${update_rate}</update_rate> <!-- Update period of accelerometer and gyroscope [s] -->
         <enable_gazebo_messages>false</enable_gazebo_messages>
-        <enable_local_ned_frame>${enable_local_ned_frame}</enable_local_ned_frame>
+        <enable_local_aaa_frame>${enable_local_aaa_frame}</enable_local_aaa_frame>
         <static_reference_frame>${reference_frame}</static_reference_frame>
       </plugin>

File: uuv_sensor_plugins/uuv_sensor_ros_plugins/urdf/magnetometer_snippets.xacro (robot description, xacro)
@@ -82,5 +82,5 @@
         <noise_amplitude>${noise_amplitude}</noise_amplitude>
         <enable_gazebo_messages>false</enable_gazebo_messages>
-        <enable_local_ned_frame>false</enable_local_ned_frame>
+        <enable_local_aaa_frame>false</enable_local_aaa_frame>
       </plugin>
     </gazebo>

File: uuv_sensor_plugins/uuv_sensor_ros_plugins/urdf/pose_3d_snippets.xacro (robot description, xacro)
@@ -14,5 +14,5 @@
 <robot xmlns:xacro="http://www.ros.org/wiki/xacro">
   <xacro:macro name="pose_3d_macro" params="namespace suffix parent_link topic
-    update_rate *origin noise_sigma reference_frame publish_ned_odom noise_amplitude">
+    update_rate *origin noise_sigma reference_frame publish_aaa_odom noise_amplitude">
     <!-- Mount a 3D pose sensor -->
     <link name="${namespace}/pose_sensor_link_${suffix}">
@@ -40,5 +40,5 @@
         <update_rate>${update_rate}</update_rate>
         <enable_gazebo_messages>false</enable_gazebo_messages>
-        <publish_ned_odom>${publish_ned_odom}</publish_ned_odom>
+        <publish_aaa_odom>${publish_aaa_odom}</publish_aaa_odom>
       </plugin>
     </gazebo>
@@ -55,5 +55,5 @@
       suffix="${suffix}"
       reference_frame="world"
-      publish_ned_odom="false">
+      publish_aaa_odom="false">
       <origin xyz="0 0 0" rpy="0 0 0" />
     </xacro:pose_3d_macro>
@@ -69,5 +69,5 @@
       suffix="default"
       reference_frame="world"
-      publish_ned_odom="false">
+      publish_aaa_odom="false">
       <origin xyz="0 0 0" rpy="0 0 0" />
     </xacro:pose_3d_macro>
@@ -83,9 +83,9 @@
       suffix="default"
       reference_frame="world"
-      publish_ned_odom="false">
+      publish_aaa_odom="false">
       <origin xyz="0 0 0" rpy="0 0 0" />
     </xacro:pose_3d_macro>
   </xacro:macro>
-  <xacro:macro name="default_pose_3d_ned" params="namespace parent_link">
+  <xacro:macro name="default_pose_3d_aaa" params="namespace parent_link">
     <xacro:pose_3d_macro
       namespace="${namespace}"
@@ -96,6 +96,6 @@
       noise_amplitude="0.0"
       suffix="default"
-      reference_frame="world_ned"
-      publish_ned_odom="true">
+      reference_frame="world_aaa"
+      publish_aaa_odom="true">
       <origin xyz="0 0 0" rpy="0 0 0" />
     </xacro:pose_3d_macro>
@@ -108,9 +108,9 @@
       </xacro:default_pose_3d_enu>
     </xacro:if>
-    <xacro:if value="${inertial_reference_frame == 'world_ned'}">
-      <xacro:default_pose_3d_ned
+    <xacro:if value="${inertial_reference_frame == 'world_aaa'}">
+      <xacro:default_pose_3d_aaa
         namespace="${namespace}"
         parent_link="${parent_link}">
-      </xacro:default_pose_3d_ned>
+      </xacro:default_pose_3d_aaa>
     </xacro:if>
   </xacro:macro>
