Commit message: FIX Path to meshes folder after refactoring
Signed-off-by: Musa Morena Marcusso Manhaes <Musa.Marcusso@de.bosch.com>

File: uuv_descriptions/urdf/rexrov_actuators.xacro (robot description, xacro)
@@ -13,5 +13,5 @@
 -->
 <robot xmlns:xacro="http://www.ros.org/wiki/xacro">
-  <xacro:property name="prop_mesh_file" value="file://$(find uuv_descriptions)/mesh/prop.dae"/>
+  <xacro:property name="prop_mesh_file" value="file://$(find uuv_descriptions)/meshes/prop.dae"/>
   <!-- Thruster joint and link snippet -->
   <xacro:macro name="thruster_macro"

File: uuv_descriptions/urdf/rexrov_base.xacro (robot description, xacro)
@@ -27,6 +27,6 @@
   <!-- Parameters -->
   <xacro:property name="namespace" value="rexrov"/>
-  <xacro:property name="visual_mesh_file" value="file://$(find uuv_descriptions)/mesh/RexROV_no_props.dae"/>
-  <xacro:property name="prop_mesh_file" value="file://$(find uuv_descriptions)/mesh/prop.dae"/>
+  <xacro:property name="visual_mesh_file" value="file://$(find uuv_descriptions)/meshes/RexROV_no_props.dae"/>
+  <xacro:property name="prop_mesh_file" value="file://$(find uuv_descriptions)/meshes/prop.dae"/>
   <!-- Mass, see p.28 in Berg2012 -->
   <xacro:property name="mass" value="1862.87"/>
